File: nixie_board/board.brd (EAGLE design)
At the start: 250 x 100 mm, 44 parts, among them IC1 74141N, IC2 74HC138D, IC3 74HC138D, U1 ATMEGA328P-AU

Commit message: [add]add toriaezu
Parts:
- added LED1: (no value), 160713 Library by matsu:1206
- added R9: (no value), 160713 Library by matsu:R3216
- added U$7: DC_JACK_2DC0005D100, 160713 Library by matsu:DC_JACK_2DC0005D100
- added U$8: PIN_HEADER_MALE_1X02_02P, 160713 Library by matsu:PIN_HEADER_MALE_1X02_02P
- moved C1 1.41 mm to (5.35, 84.1)
- moved U$2 0.77 mm to (5.65, 93.7), turned to 270 degrees
Connections:
- new net N$16: LED1.A, R9.1
- net +5V: now also R9.2, U$7.1
- net 200V: now also U$8.P$1
- net GND: now also LED1.C, U$7.2, U$7.3, U$8.P$2
Changed lines of the file:
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@@
 </class>
 </classes>
-<designrules name="default *">
+<designrules name="Elecrow_2-layer_eagle_rule">
 <description language="de">&lt;b&gt;EAGLE Design Rules&lt;/b&gt;
 &lt;p&gt;
@@
 necessary adjustments and save your customized
 design rules under a new name.</description>
-<description language="zh">&lt;b&gt;Elecrow PCB EAGLE Design Rules&lt;/b&gt;
+<description language="zh">&lt;b&gt;Elecrow EAGLE Design Rules&lt;/b&gt;
 </description>
 <param name="layerSetup" value="(1*16)"/>
 <param name="mtCopper" value="0.035mm 0.035mm 0.035mm 0.035mm 0.035mm 0.035mm 0.035mm 0.035mm 0.035mm 0.035mm 0.035mm 0.035mm 0.035mm 0.035mm 0.035mm 0.035mm"/>
-<param name="mtIsolate" value="1.6mm 1.2mm 0.2mm 0.15mm 0.2mm 0.15mm 0.2mm 0.15mm 0.2mm 0.15mm 0.2mm 0.15mm 0.2mm 0.15mm 0.2mm"/>
+<param name="mtIsolate" value="1.5mm 0.15mm 0.2mm 0.15mm 0.2mm 0.15mm 0.2mm 0.15mm 0.2mm 0.15mm 0.2mm 0.15mm 0.2mm 0.15mm 0.2mm"/>
 <param name="mdWireWire" value="6mil"/>
-<param name="mdWirePad" value="8mil"/>
+<param name="mdWirePad" value="6mil"/>
 <param name="mdWireVia" value="6mil"/>
-<param name="mdPadPad" value="12mil"/>
-<param name="mdPadVia" value="8mil"/>
-<param name="mdViaVia" value="12mil"/>
+<param name="mdPadPad" value="6mil"/>
+<param name="mdPadVia" value="6mil"/>
+<param name="mdViaVia" value="6mil"/>
 <param name="mdSmdPad" value="0mil"/>
 <param name="mdSmdVia" value="0mil"/>
@@
 <param name="mdViaViaSameLayer" value="8mil"/>
 <param name="mnLayersViaInSmd" value="2"/>
-<param name="mdCopperDimension" value="20mil"/>
+<param name="mdCopperDimension" value="10mil"/>
 <param name="mdDrill" value="10mil"/>
 <param name="mdSmdStop" value="0mil"/>
@@
 <param name="rvMicroViaOuter" value="0.25"/>
 <param name="rvMicroViaInner" value="0.25"/>
-<param name="rlMinPadTop" value="6mil"/>
+<param name="rlMinPadTop" value="10mil"/>
 <param name="rlMaxPadTop" value="20mil"/>
-<param name="rlMinPadInner" value="6mil"/>
+<param name="rlMinPadInner" value="10mil"/>
 <param name="rlMaxPadInner" value="20mil"/>
-<param name="rlMinPadBottom" value="6mil"/>
+<param name="rlMinPadBottom" value="10mil"/>
 <param name="rlMaxPadBottom" value="20mil"/>
 <param name="rlMinViaOuter" value="6mil"/>
@@
 <param name="mvStopFrame" value="1"/>
 <param name="mvCreamFrame" value="0"/>
-<param name="mlMinStopFrame" value="0mil"/>
-<param name="mlMaxStopFrame" value="0mil"/>
+<param name="mlMinStopFrame" value="2mil"/>
+<param name="mlMaxStopFrame" value="2mil"/>
 <param name="mlMinCreamFrame" value="0mil"/>
 <param name="mlMaxCreamFrame" value="0mil"/>
@@
 </element>
 <element name="U$1" library="con-hirose" package="ZX62R-B-5P" value="MICRO-USB-ZX62R-B-5P" x="27.94" y="97.79" rot="R270"/>
-<element name="U$2" library="crystals" package="FA-238" value="FA-238" x="6.35" y="93.345" rot="R90"/>
+<element name="U$2" library="crystals" package="FA-238" value="FA-238" x="5.65" y="93.655" rot="R270"/>
 <element name="IC1" library="74xx-eu" library_urn="urn:adsk.eagle:library:85" package="DIL16" package3d_urn="urn:adsk.eagle:package:2009/1" value="74141N" x="25.4" y="72.39" rot="R180"/>
 <element name="IC2" library="74xx-eu" library_urn="urn:adsk.eagle:library:85" package="SO16" package3d_urn="urn:adsk.eagle:package:2010/1" value="74HC138D" x="26.67" y="83.82"/>
@@
 <element name="N9" library="russian-nixies" package="IN-19" value="IN-19A" x="95.93" y="23.56" rot="R90"/>
 <element name="N10" library="russian-nixies" package="IN-19" value="IN-19B" x="112.44" y="23.56" rot="R90"/>
-<element name="C1" library="160713 Library by matsu" package="E5-8,5" value="" x="6.35" y="85.09" rot="R270"/>
+<element name="C1" library="160713 Library by matsu" package="E5-8,5" value="" x="5.35" y="84.09" rot="R270"/>
 <element name="RESET" library="160713 Library by matsu" package="DTS6" value="DTS-6" x="6.35" y="73.66" rot="R90"/>
 <element name="R10" library="160713 Library by matsu" package="R3216" value="" x="12.7" y="80.01"/>
+<element name="U$7" library="160713 Library by matsu" package="DC_JACK_2DC0005D100" value="DC_JACK_2DC0005D100" x="10" y="62" rot="R180"/>
+<element name="LED1" library="160713 Library by matsu" package="1206" value="" x="7" y="50"/>
+<element name="R9" library="160713 Library by matsu" package="R3216" value="" x="6" y="45"/>
+<element name="U$8" library="160713 Library by matsu" package="PIN_HEADER_MALE_1X02_02P" value="PIN_HEADER_MALE_1X02_02P" x="6" y="36" rot="R90"/>
 </elements>
 <signals>
@@
 <contactref element="RESET" pad="1"/>
 <contactref element="RESET" pad="2"/>
+<contactref element="U$7" pad="3"/>
+<contactref element="U$7" pad="2"/>
+<contactref element="LED1" pad="C"/>
+<contactref element="U$8" pad="P$2"/>
 <wire x1="100.33" y1="81.28" x2="105.41" y2="81.28" width="0" layer="19" extent="1-1"/>
 <wire x1="45.085" y1="80.7466" x2="100.33" y2="81.28" width="0" layer="19" extent="1-1"/>
@@
 <wire x1="10.9982" y1="91.3638" x2="19.4818" y2="90.5764" width="0" layer="19" extent="1-1"/>
 <wire x1="10.9982" y1="89.7636" x2="10.9982" y2="91.3638" width="0" layer="19" extent="1-1"/>
-<wire x1="6.35" y1="93.345" x2="10.9982" y2="91.3638" width="0" layer="19" extent="1-1"/>
-<wire x1="7.95" y1="95.545" x2="6.35" y2="93.345" width="0" layer="19" extent="1-1"/>
-<wire x1="6.35" y1="82.55" x2="10.9982" y2="89.7636" width="0" layer="19" extent="1-1"/>
-<wire x1="4.0894" y1="76.9112" x2="6.35" y2="82.55" width="0" layer="19" extent="1-1"/>
+<wire x1="5.65" y1="93.655" x2="10.9982" y2="91.3638" width="0" layer="19" extent="1-1"/>
+<wire x1="4.05" y1="91.455" x2="5.65" y2="93.655" width="0" layer="19" extent="1-1"/>
+<wire x1="5.35" y1="81.55" x2="10.9982" y2="89.7636" width="0" layer="19" extent="1-1"/>
+<wire x1="4.0894" y1="76.9112" x2="5.35" y2="81.55" width="0" layer="19" extent="1-1"/>
 <wire x1="4.0894" y1="70.4088" x2="4.0894" y2="76.9112" width="0" layer="19" extent="1-1"/>
 <wire x1="29.24" y1="95.115" x2="19.4818" y2="90.5764" width="0" layer="19" extent="1-1"/>
 <wire x1="24.13" y1="68.58" x2="27.305" y2="80.7466" width="0" layer="19" extent="1-1"/>
+<wire x1="10" y1="57.2" x2="24.13" y2="68.58" width="0" layer="19" extent="1-1"/>
+<wire x1="7" y1="62" x2="10" y2="57.2" width="0" layer="19" extent="1-1"/>
+<wire x1="8.422" y1="50" x2="7" y2="62" width="0" layer="19" extent="1-1"/>
+<wire x1="6" y1="37.27" x2="8.422" y2="50" width="0" layer="19" extent="1-1"/>
 </signal>
 <signal name="+5V">
@@
 <wire x1="107.95" y1="95.38" x2="102.365" y2="95.38" width="0.4064" layer="1"/>
 <wire x1="102.365" y1="95.38" x2="102.235" y2="95.25" width="0.4064" layer="1"/>
+<contactref element="U$7" pad="1"/>
+<contactref element="R9" pad="2"/>
 <wire x1="102.365" y1="95.38" x2="102.87" y2="95.38" width="0" layer="19" extent="1-1"/>
 <wire x1="94.615" y1="95.25" x2="102.235" y2="95.25" width="0" layer="19" extent="1-1"/>
@@
 <wire x1="10.9982" y1="88.9762" x2="19.4818" y2="88.1634" width="0" layer="19" extent="1-1"/>
 <wire x1="10.9982" y1="90.5764" x2="10.9982" y2="88.9762" width="0" layer="19" extent="1-1"/>
-<wire x1="6.35" y1="87.63" x2="10.9982" y2="88.9762" width="0" layer="19" extent="1-1"/>
+<wire x1="5.35" y1="86.63" x2="10.9982" y2="88.9762" width="0" layer="19" extent="1-1"/>
 <wire x1="28.575" y1="80.7466" x2="22.225" y2="86.8934" width="0" layer="19" extent="1-1"/>
 <wire x1="24.13" y1="76.2" x2="28.575" y2="80.7466" width="0" layer="19" extent="1-1"/>
 <wire x1="14.1" y1="80.01" x2="10.9982" y2="88.9762" width="0" layer="19" extent="1-1"/>
+<wire x1="13.1" y1="62" x2="24.13" y2="76.2" width="0" layer="19" extent="1-1"/>
+<wire x1="7.4" y1="45" x2="13.1" y2="62" width="0" layer="19" extent="1-1"/>
 </signal>
 <signal name="N$1">
 <contactref element="U$2" pad="3"/>
 <contactref element="U1" pad="7"/>
-<wire x1="10.9982" y1="88.1634" x2="6.35" y2="95.545" width="0" layer="19" extent="1-1"/>
+<wire x1="10.9982" y1="88.1634" x2="5.65" y2="91.455" width="0" layer="19" extent="1-1"/>
 </signal>
 <signal name="N$2">
 <contactref element="U$2" pad="1"/>
 <contactref element="U1" pad="8"/>
-<wire x1="10.9982" y1="87.376" x2="7.95" y2="93.345" width="0" layer="19" extent="1-1"/>
+<wire x1="10.9982" y1="87.376" x2="4.05" y2="93.655" width="0" layer="19" extent="1-1"/>
 </signal>
 <signal name="VCC">
@@
 <wire x1="88.9" y1="74.8" x2="93.98" y2="74.8" width="0.4064" layer="1"/>
 <wire x1="118.11" y1="74.8" x2="113.03" y2="74.8" width="0.4064" layer="1"/>
+<contactref element="U$8" pad="P$1"/>
 <wire x1="93.98" y1="74.8" x2="113.03" y2="74.8" width="0" layer="19" extent="1-1"/>
 <wire x1="69.85" y1="74.8" x2="78.74" y2="74.8" width="0" layer="19" extent="1-1"/>
+<wire x1="6" y1="34.73" x2="54.61" y2="74.8" width="0" layer="19" extent="1-1"/>
 </signal>
 <signal name="N$11">
@@
 <wire x1="8.6106" y1="70.4088" x2="8.6106" y2="76.9112" width="0" layer="19" extent="1-1"/>
 </signal>
+<signal name="N$16">
+<contactref element="LED1" pad="A"/>
+<contactref element="R9" pad="1"/>
+<wire x1="5.578" y1="50" x2="4.6" y2="45" width="0" layer="19" extent="1-1"/>
+</signal>
 </signals>
