File: nixie_board/board.brd (EAGLE design)
At the start: 240 x 50 mm, 18 parts

Commit message: [add]add all
Parts:
- removed LED1, LED2, LED3, LED4, LED5, LED6, LED7, LED8: WS2812B_5050N, adafruit:WS2812B-NARROW
Connections:
- removed net N$1: LED1.2-DOUT, LED2.4-DIN
- removed net N$2: LED2.2-DOUT, LED3.4-DIN
- removed net N$3: LED3.2-DOUT, LED4.4-DIN
- removed net N$4: LED4.2-DOUT, LED5.4-DIN
- removed net N$5: LED5.2-DOUT, LED6.4-DIN
- removed net N$6: LED6.2-DOUT, LED7.4-DIN
- removed net N$7: LED7.2-DOUT, LED8.4-DIN
- net +5V: no longer LED1.1-VDD, LED2.1-VDD, LED3.1-VDD, LED4.1-VDD, LED5.1-VDD, LED6.1-VDD, LED7.1-VDD, LED8.1-VDD
- net GND: no longer LED1.3-GND, LED2.3-GND, LED3.3-GND, LED4.3-GND, LED5.3-GND, LED6.3-GND, LED7.3-GND, LED8.3-GND
- net N$8: no longer LED1.4-DIN
Routing:
- net N$6: track 59.8 -> 0.00 mm, vias 2 -> 0
- net N$7: track 50.2 -> 0.00 mm, vias 2 -> 0
- net N$5: track 49.9 -> 0.00 mm, vias 2 -> 0
- net N$3: track 49.0 -> 0.00 mm, vias 2 -> 0
- net N$2: track 48.4 -> 0.00 mm, vias 2 -> 0
- net N$1: track 47.8 -> 0.00 mm, vias 2 -> 0
- net N$4: track 45.3 -> 0.00 mm, vias 2 -> 0
- net GND: track 349.4 -> 339.7 mm
- net +5V: track 330.6 -> 324.0 mm
- net N$8: track 106.1 -> 103.8 mm
