File: nixie_board/board.sch (EAGLE design)
At the start: 44 parts, among them IC1 74141N, IC2 74HC138D, IC3 74HC138D, U1 ATMEGA328P-AU

Commit message: [add]add toriaezu
Parts:
- added LED1: (no value), 160713 Library by matsu:LEDSMT1206
- added R9: (no value), 160713 Library by matsu:R-EU_R3216
- added U$7: DC_JACK_2DC0005D100, 160713 Library by matsu:DC_JACK_2DC0005D100
- added U$8: PIN_HEADER_MALE_1X02_02P, 160713 Library by matsu:PIN_HEADER_MALE_1X02_02P
Connections:
- new net N$16: LED1.A, R9.1
- net +5V: now also R9.2, U$7.1
- net 200V: now also U$8.1
- net GND: now also LED1.C, U$7.2, U$7.3, U$8.2
Other:
- moved on the sheet: C1
Changed lines of the file:
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@@
 <part name="R10" library="160713 Library by matsu" deviceset="R-EU_" device="R3216"/>
 <part name="P+12" library="160713 Library by matsu" deviceset="+5V" device=""/>
+<part name="U$7" library="160713 Library by matsu" deviceset="DC_JACK_2DC0005D100" device=""/>
+<part name="P+21" library="160713 Library by matsu" deviceset="+5V" device=""/>
+<part name="GND13" library="160713 Library by matsu" deviceset="GND" device=""/>
+<part name="P+22" library="160713 Library by matsu" deviceset="+5V" device=""/>
+<part name="GND14" library="160713 Library by matsu" deviceset="GND" device=""/>
+<part name="LED1" library="160713 Library by matsu" deviceset="LED" device="SMT1206"/>
+<part name="R9" library="160713 Library by matsu" deviceset="R-EU_" device="R3216"/>
+<part name="U$8" library="160713 Library by matsu" deviceset="PIN_HEADER_MALE_1X02_02P" device=""/>
+<part name="GND15" library="160713 Library by matsu" deviceset="GND" device=""/>
 </parts>
 <sheets>
@@
 <instance part="GND8" gate="1" x="228.6" y="-137.16"/>
 <instance part="P+9" gate="1" x="45.72" y="-15.24"/>
-<instance part="GND9" gate="1" x="45.72" y="-43.18"/>
-<instance part="C1" gate="G$1" x="45.72" y="-27.94"/>
+<instance part="GND9" gate="1" x="45.72" y="-45.72"/>
+<instance part="C1" gate="G$1" x="45.72" y="-30.48"/>
 <instance part="IC2" gate="P" x="132.08" y="101.6" rot="R90"/>
 <instance part="IC3" gate="P" x="132.08" y="63.5" rot="R90"/>
@@
 <instance part="R10" gate="G$1" x="93.98" y="66.04" rot="R90"/>
 <instance part="P+12" gate="1" x="93.98" y="76.2"/>
+<instance part="U$7" gate="G$1" x="-7.62" y="-7.62"/>
+<instance part="P+21" gate="1" x="2.54" y="0"/>
+<instance part="GND13" gate="1" x="2.54" y="-15.24"/>
+<instance part="P+22" gate="1" x="58.42" y="-15.24"/>
+<instance part="GND14" gate="1" x="58.42" y="-45.72"/>
+<instance part="LED1" gate="G$1" x="58.42" y="-35.56"/>
+<instance part="R9" gate="G$1" x="58.42" y="-25.4" rot="R90"/>
+<instance part="U$8" gate="G$1" x="27.94" y="-3.81" rot="R270"/>
+<instance part="GND15" gate="1" x="40.64" y="-10.16"/>
 </instances>
 <busses>
@@
 <pinref part="C1" gate="G$1" pin="-"/>
 <pinref part="GND9" gate="1" pin="GND"/>
-<wire x1="45.72" y1="-33.02" x2="45.72" y2="-40.64" width="0.1524" layer="91"/>
+<wire x1="45.72" y1="-35.56" x2="45.72" y2="-43.18" width="0.1524" layer="91"/>
 </segment>
 <segment>
@@
 <pinref part="RESET" gate="G$1" pin="S1"/>
 <wire x1="91.44" y1="43.18" x2="91.44" y2="45.72" width="0.1524" layer="91"/>
+</segment>
+<segment>
+<pinref part="U$7" gate="G$1" pin="3"/>
+<wire x1="-2.54" y1="-7.62" x2="2.54" y2="-7.62" width="0.1524" layer="91"/>
+<wire x1="2.54" y1="-7.62" x2="2.54" y2="-10.16" width="0.1524" layer="91"/>
+<pinref part="U$7" gate="G$1" pin="2"/>
+<wire x1="2.54" y1="-10.16" x2="-2.54" y2="-10.16" width="0.1524" layer="91"/>
+<pinref part="GND13" gate="1" pin="GND"/>
+<wire x1="2.54" y1="-10.16" x2="2.54" y2="-12.7" width="0.1524" layer="91"/>
+<junction x="2.54" y="-10.16"/>
+</segment>
+<segment>
+<pinref part="GND14" gate="1" pin="GND"/>
+<pinref part="LED1" gate="G$1" pin="C"/>
+<wire x1="58.42" y1="-43.18" x2="58.42" y2="-40.64" width="0.1524" layer="91"/>
+</segment>
+<segment>
+<pinref part="U$8" gate="G$1" pin="2"/>
+<pinref part="GND15" gate="1" pin="GND"/>
+<wire x1="33.02" y1="-5.08" x2="40.64" y2="-5.08" width="0.1524" layer="91"/>
+<wire x1="40.64" y1="-5.08" x2="40.64" y2="-7.62" width="0.1524" layer="91"/>
 </segment>
 </net>
@@
 <pinref part="P+9" gate="1" pin="+5V"/>
 <pinref part="C1" gate="G$1" pin="+"/>
-<wire x1="45.72" y1="-17.78" x2="45.72" y2="-25.4" width="0.1524" layer="91"/>
+<wire x1="45.72" y1="-17.78" x2="45.72" y2="-27.94" width="0.1524" layer="91"/>
 </segment>
 <segment>
@@
 <pinref part="P+12" gate="1" pin="+5V"/>
 <wire x1="93.98" y1="71.12" x2="93.98" y2="73.66" width="0.1524" layer="91"/>
+</segment>
+<segment>
+<pinref part="U$7" gate="G$1" pin="1"/>
+<wire x1="-2.54" y1="-5.08" x2="2.54" y2="-5.08" width="0.1524" layer="91"/>
+<pinref part="P+21" gate="1" pin="+5V"/>
+<wire x1="2.54" y1="-2.54" x2="2.54" y2="-5.08" width="0.1524" layer="91"/>
+</segment>
+<segment>
+<pinref part="P+22" gate="1" pin="+5V"/>
+<pinref part="R9" gate="G$1" pin="2"/>
+<wire x1="58.42" y1="-20.32" x2="58.42" y2="-17.78" width="0.1524" layer="91"/>
 </segment>
 </net>
@@
 <pinref part="R30" gate="G$1" pin="2"/>
 <wire x1="241.3" y1="-81.28" x2="246.38" y2="-81.28" width="0.1524" layer="91"/>
+</segment>
+<segment>
+<pinref part="U$8" gate="G$1" pin="1"/>
+<wire x1="33.02" y1="-2.54" x2="40.64" y2="-2.54" width="0.1524" layer="91"/>
+<wire x1="40.64" y1="0" x2="40.64" y2="-2.54" width="0.1524" layer="91"/>
+<label x="40.64" y="0" size="1.778" layer="95" rot="R90" xref="yes"/>
 </segment>
 </net>
@@
 </segment>
 </net>
+<net name="N$16" class="0">
+<segment>
+<pinref part="LED1" gate="G$1" pin="A"/>
+<pinref part="R9" gate="G$1" pin="1"/>
+<wire x1="58.42" y1="-30.48" x2="58.42" y2="-33.02" width="0.1524" layer="91"/>
+</segment>
+</net>
