File: nixie_board/board.sch (EAGLE design)
At the start: 44 parts, among them IC1 74141N, IC2 74HC138D, IC3 74HC138D, U1 ATMEGA328P-AU

Commit message: [add]iroiro
Parts:
- removed U1: ATMEGA328P-AU, Atmel-ATMEGA328P-AU:ATMEGA328P-AU
- added C2, C3: (no value), 160713 Library by matsu:CPOL-EUE2.5-6
- added IC4: LT1963ES8-3.3, linear-technology:LT1963ES8-3.3
- added IC5: FT232RL, ftdichip:FT232RL
- added U$4: DC_JACK_2DC0005D100, 160713 Library by matsu:DC_JACK_2DC0005D100
- added U2: ESP-WROOM-32, esp32:ESP-WROOM-32
- U$2: value FA-238 -> PIN_HEADER_MALE_1X08_08P; device crystals:FA-238 -> 160713 Library by matsu:PIN_HEADER_MALE_1X08_08P
Connections:
- new net +3V3: C2.+, IC1P.VCC, IC2P.VCC, IC4G$1.OUT, IC4G$1.SENSE, R10.2, U2.3V3
- new net N$16: U2.EN
- net +5V: now also C3.+, IC4G$1.!SHDN, IC4G$1.IN; no longer IC1P.VCC, IC2A.G1, IC2P.VCC, R10.2, U1.AVCC, U1.VCC, U1.VCC_2
- net GND: now also C2.-, C3.-, IC3P.GND, IC4G$1.GND, U2.GND, U2.GND@1, U2.GND@15, U2.GND@38; no longer U$2.GND_2, U$2.GND_4, U1.GND, U1.GND_2, U1.GND_3
- net LHDP: no longer U1.PD3
- net N$1: now also IC2A.G1; no longer U$2.XTALOUT, U1.PB6
- net N$15: no longer U1.PC6
- net N$2: now also IC3P.VCC; no longer U$2.XTALIN, U1.PB7
- net N$3: now also U2.IO14; no longer U1.PD7
- net N$4: now also U2.IO27; no longer U1.PD6
- net N$5: now also U2.IO26; no longer U1.PD5
- net N$6: now also U2.IO25; no longer U1.PD4
- net NIX1: now also U2.IO33; no longer U1.PC3
- net NIX2: now also U2.IO32; no longer U1.PC2
- net NIX3: now also U2.IO35; no longer U1.PC1
- net NIX4: now also U2.IO34; no longer U1.PC0
- net RHDP: no longer U1.PD2
- net RXI: no longer U1.PD0
- net TXO: no longer U1.PD1
Other:
- moved on the sheet: C1, R10, RESET, U$1

Commit message: [add]complete
Parts:
- removed C1: (no value), 160713 Library by matsu:CPOL-EUE5-8.5
- removed C2, C3: (no value), 160713 Library by matsu:CPOL-EUE2.5-6
- removed IC1: 74141N, 74xx-eu:74141N
- removed IC2, IC3: 74HC138D, 74xx-eu:74HC138D
- removed IC4: LT1963ES8-3.3, linear-technology:LT1963ES8-3.3
- removed IC5: FT232RL, ftdichip:FT232RL
- removed N10: IN-19B, russian-nixies:IN-19B
- removed N9: IN-19A, russian-nixies:IN-19A
- removed R1, R17, R18, R19, R2, R20, R21, R22, R23, R24, R25, R26, R27, R28, R29, R3, R30, R4, R5, R6, R7, R8: (no value), resistor:R-EU_M3216
- removed R10: (no value), 160713 Library by matsu:R-EU_R3216
- removed RESET: DTS-6, 160713 Library by matsu:DTS-6
- removed U$3, U$5, U$6: TLP627-4, 160713 Library by matsu:TLP627-4
- removed U$4: DC_JACK_2DC0005D100, 160713 Library by matsu:DC_JACK_2DC0005D100
- removed U2: ESP-WROOM-32, esp32:ESP-WROOM-32
- added LED1, LED2, LED3, LED4, LED5, LED6, LED7, LED8: WS2812B_5050N, adafruit:WS2812B_5050N
- U$1: value MICRO-USB-ZX62R-B-5P -> PIN_HEADER_MALE_2X10_20P; device con-hirose:MICRO-USB-ZX62R-B-5P -> 160713 Library by matsu:PIN_HEADER_MALE_2X10_20P
- U$2: value PIN_HEADER_MALE_1X08_08P -> PIN_HEADER_MALE_1X03_03P; device 160713 Library by matsu:PIN_HEADER_MALE_1X08_08P -> 160713 Library by matsu:PIN_HEADER_MALE_1X03_03P
Connections:
- removed net +3V3: C2.+, IC1P.VCC, IC2P.VCC, IC4G$1.OUT, IC4G$1.SENSE, R10.2, U2.3V3
- removed net 200V: R21.2, R22.2, R23.2, R24.2, R29.2, R30.2, R5.2, R6.2, R7.2, R8.2
- removed net ANODE0: IC2A.Y0, U$3.P$2
- removed net ANODE1: IC2A.Y1, U$3.P$4
- removed net ANODE10: IC3A.Y2
- removed net ANODE11: IC3A.Y3
- removed net ANODE12: IC3A.Y4
- removed net ANODE13: IC3A.Y5
- removed net ANODE14: IC3A.Y6
- removed net ANODE15: IC3A.Y7
- removed net ANODE2: IC2A.Y2, U$3.P$6
- removed net ANODE3: IC2A.Y3, U$3.P$8
- removed net ANODE4: IC2A.Y5, U$5.P$2
- removed net ANODE5: IC2A.Y4, U$5.P$4
- removed net ANODE6: IC2A.Y6, U$5.P$6
- removed net ANODE7: IC2A.Y7, U$5.P$8
- removed net ANODE8: IC3A.Y0, U$6.P$2
- removed net ANODE9: IC3A.Y1, U$6.P$4
- removed net DTR: U$1.1
- removed net LHDP: U$6.P$6
- removed net N$10: R4.2, U$3.P$7
- removed net N$11: R8.1, U$3.P$10
- removed net N$12: R7.1, U$3.P$12
- removed net N$13: R6.1, U$3.P$14
- removed net N$14: R5.1, U$3.P$16
- removed net N$15: R10.1, RESET.P, RESET.P1
- removed net N$16: U2.EN
- removed net N$23: R17.2, U$5.P$1
- removed net N$24: R18.2, U$5.P$3
- removed net N$25: R19.2, U$5.P$5
- removed net N$26: R20.2, U$5.P$7
- removed net N$27: R24.1, U$5.P$10
- removed net N$28: R23.1, U$5.P$12
- removed net N$29: R22.1, U$5.P$14
- removed net N$30: R21.1, U$5.P$16
- removed net N$31: R25.2, U$6.P$1
- removed net N$32: R26.2, U$6.P$3
- removed net N$33: R27.2, U$6.P$5
- removed net N$34: R28.2, U$6.P$7
- removed net N$37: R30.1, U$6.P$14
- removed net N$38: R29.1, U$6.P$16
- removed net N$9: R3.2, U$3.P$5
- removed net NIX1: IC2A.A, IC3A.A, U2.IO33
- removed net NIX2: IC2A.B, IC3A.B, U2.IO32
- removed net NIX3: IC2A.C, IC3A.C, U2.IO35
- removed net NIX4: IC2A.G2A, IC3A.G1, U2.IO34
- removed net NIXIE_ANODE10: N10.A, U$6.P$13
- removed net NIXIE_ANODE9: N9.A, U$6.P$15
- removed net RHDP: U$6.P$8
- removed net RXI: U$1.3
- removed net TXO: U$1.2
- net +5V: now also LED1.VDD, LED2.VDD, LED3.VDD, LED4.VDD, LED5.VDD, LED6.VDD, LED7.VDD, LED8.VDD, U$2.1; no longer C1.+, C3.+, IC4G$1.!SHDN, IC4G$1.IN, R1.1, R17.1, R18.1, R19.1, R2.1, R20.1, R25.1, R26.1, R27.1, R28.1, R3.1, R4.1, U$1.4
- net DOT0: now also U$1.P$3; no longer U$6.P$12
- net DOT1: now also U$1.P$1; no longer U$6.P$10
- net GND: now also LED1.GND, LED2.GND, LED3.GND, LED4.GND, LED5.GND, LED6.GND, LED7.GND, LED8.GND, U$2.2; no longer C1.-, C2.-, C3.-, IC1P.GND, IC2A.G2B, IC2P.GND, IC3A.G2A, IC3A.G2B, IC3P.GND, IC4G$1.GND, RESET.S, RESET.S1, U$1.5, U$6.P$11, U$6.P$9, U2.GND, U2.GND@1, U2.GND@15, U2.GND@38
- net N$1: now also LED1.DO, LED2.DI; no longer IC2A.G1
- net N$2: now also LED2.DO, LED3.DI; no longer IC3P.VCC
- net N$3: now also LED3.DO, LED4.DI; no longer IC1A.A, U2.IO14
- net N$4: now also LED4.DO, LED5.DI; no longer IC1A.B, U2.IO27
- net N$5: now also LED5.DO, LED6.DI; no longer IC1A.C, U2.IO26
- net N$6: now also LED6.DO, LED7.DI; no longer IC1A.D, U2.IO25
- net N$7: now also LED7.DO, LED8.DI; no longer R1.2, U$3.P$1
- net N$8: now also LED1.DI, U$2.3; no longer R2.2, U$3.P$3
- net NIXIE0: now also U$1.P$20; no longer IC1A.0, N10.P$1, N9.P$1
- net NIXIE1: now also U$1.P$18; no longer N10.P$2, N9.P$2
- net NIXIE2: now also U$1.P$16; no longer IC1A.1, IC1A.2, N10.P$3, N9.P$3
- net NIXIE3: now also U$1.P$14; no longer IC1A.3, N10.P$4, N9.P$4
- net NIXIE4: now also U$1.P$12; no longer IC1A.4, N10.P$5, N9.P$5
- net NIXIE5: now also U$1.P$10; no longer IC1A.5, N10.P$6, N9.P$6
- net NIXIE6: now also U$1.P$8; no longer IC1A.6, N10.P$7, N9.P$7
- net NIXIE7: now also U$1.P$6; no longer IC1A.7, N10.P$8, N9.P$8
- net NIXIE8: now also U$1.P$4; no longer IC1A.8
- net NIXIE9: now also U$1.P$2; no longer IC1A.9
- net NIXIE_ANODE1: now also U$1.P$5; no longer U$3.P$15
- net NIXIE_ANODE2: now also U$1.P$7; no longer U$3.P$13
- net NIXIE_ANODE3: now also U$1.P$9; no longer U$3.P$11
- net NIXIE_ANODE4: now also U$1.P$11; no longer U$3.P$9
- net NIXIE_ANODE5: now also U$1.P$13; no longer U$5.P$15
- net NIXIE_ANODE6: now also U$1.P$15; no longer U$5.P$13
- net NIXIE_ANODE7: now also U$1.P$17; no longer U$5.P$11
- net NIXIE_ANODE8: now also U$1.P$19; no longer U$5.P$9

Commit message: [add]add all
Parts:
- removed LED1, LED2, LED3, LED4, LED5, LED6, LED7, LED8: WS2812B_5050N, adafruit:WS2812B_5050N
Connections:
- removed net N$1: LED1.DO, LED2.DI
- removed net N$2: LED2.DO, LED3.DI
- removed net N$3: LED3.DO, LED4.DI
- removed net N$4: LED4.DO, LED5.DI
- removed net N$5: LED5.DO, LED6.DI
- removed net N$6: LED6.DO, LED7.DI
- removed net N$7: LED7.DO, LED8.DI
- net +5V: no longer LED1.VDD, LED2.VDD, LED3.VDD, LED4.VDD, LED5.VDD, LED6.VDD, LED7.VDD, LED8.VDD
- net GND: no longer LED1.GND, LED2.GND, LED3.GND, LED4.GND, LED5.GND, LED6.GND, LED7.GND, LED8.GND
- net N$8: no longer LED1.DI
Changed lines of the file:
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@@
 <?xml version="1.0" encoding="utf-8"?>
 <!DOCTYPE eagle SYSTEM "eagle.dtd">
-<eagle version="8.5.2">
+<eagle version="9.1.2">
 <drawing>
 <settings>
@@
 <part name="N7" library="russian-nixies" deviceset="IN-14" device=""/>
 <part name="N8" library="russian-nixies" deviceset="IN-14" device=""/>
-<part name="LED1" library="adafruit" library_urn="urn:adsk.eagle:library:420" deviceset="WS2812B" device="_5050N"/>
-<part name="LED2" library="adafruit" library_urn="urn:adsk.eagle:library:420" deviceset="WS2812B" device="_5050N"/>
-<part name="LED3" library="adafruit" library_urn="urn:adsk.eagle:library:420" deviceset="WS2812B" device="_5050N"/>
-<part name="LED4" library="adafruit" library_urn="urn:adsk.eagle:library:420" deviceset="WS2812B" device="_5050N"/>
-<part name="LED5" library="adafruit" library_urn="urn:adsk.eagle:library:420" deviceset="WS2812B" device="_5050N"/>
-<part name="LED6" library="adafruit" library_urn="urn:adsk.eagle:library:420" deviceset="WS2812B" device="_5050N"/>
-<part name="LED7" library="adafruit" library_urn="urn:adsk.eagle:library:420" deviceset="WS2812B" device="_5050N"/>
-<part name="LED8" library="adafruit" library_urn="urn:adsk.eagle:library:420" deviceset="WS2812B" device="_5050N"/>
 <part name="P+1" library="160713 Library by matsu" deviceset="+5V" device=""/>
 <part name="P+2" library="160713 Library by matsu" deviceset="+5V" device=""/>
@@
 <instance part="N7" gate="G$1" x="406.4" y="33.02" rot="R90"/>
 <instance part="N8" gate="G$1" x="454.66" y="33.02" rot="R90"/>
-<instance part="LED1" gate="G$1" x="297.18" y="-22.86"/>
-<instance part="LED2" gate="G$1" x="322.58" y="-22.86"/>
-<instance part="LED3" gate="G$1" x="347.98" y="-22.86"/>
-<instance part="LED4" gate="G$1" x="373.38" y="-22.86"/>
-<instance part="LED5" gate="G$1" x="398.78" y="-22.86"/>
-<instance part="LED6" gate="G$1" x="424.18" y="-22.86"/>
-<instance part="LED7" gate="G$1" x="449.58" y="-22.86"/>
-<instance part="LED8" gate="G$1" x="474.98" y="-22.86"/>
 <instance part="P+1" gate="1" x="302.26" y="-5.08"/>
 <instance part="P+2" gate="1" x="327.66" y="-5.08"/>
@@
 </segment>
 </net>
-<net name="N$1" class="0">
-<segment>
-<pinref part="LED1" gate="G$1" pin="DO"/>
-<pinref part="LED2" gate="G$1" pin="DI"/>
-</segment>
-</net>
-<net name="N$2" class="0">
-<segment>
-<pinref part="LED2" gate="G$1" pin="DO"/>
-<pinref part="LED3" gate="G$1" pin="DI"/>
-</segment>
-</net>
-<net name="N$3" class="0">
-<segment>
-<pinref part="LED3" gate="G$1" pin="DO"/>
-<pinref part="LED4" gate="G$1" pin="DI"/>
-</segment>
-</net>
-<net name="N$4" class="0">
-<segment>
-<pinref part="LED4" gate="G$1" pin="DO"/>
-<pinref part="LED5" gate="G$1" pin="DI"/>
-</segment>
-</net>
-<net name="N$5" class="0">
-<segment>
-<pinref part="LED5" gate="G$1" pin="DO"/>
-<pinref part="LED6" gate="G$1" pin="DI"/>
-</segment>
-</net>
-<net name="N$6" class="0">
-<segment>
-<pinref part="LED6" gate="G$1" pin="DO"/>
-<pinref part="LED7" gate="G$1" pin="DI"/>
-</segment>
-</net>
-<net name="N$7" class="0">
-<segment>
-<pinref part="LED7" gate="G$1" pin="DO"/>
-<pinref part="LED8" gate="G$1" pin="DI"/>
-</segment>
-</net>
 <net name="+5V" class="0">
-<segment>
-<pinref part="LED1" gate="G$1" pin="VDD"/>
-<pinref part="P+1" gate="1" pin="+5V"/>
-</segment>
-<segment>
-<pinref part="LED2" gate="G$1" pin="VDD"/>
-<pinref part="P+2" gate="1" pin="+5V"/>
-</segment>
-<segment>
-<pinref part="LED3" gate="G$1" pin="VDD"/>
-<pinref part="P+3" gate="1" pin="+5V"/>
-</segment>
-<segment>
-<pinref part="LED4" gate="G$1" pin="VDD"/>
-<pinref part="P+4" gate="1" pin="+5V"/>
-</segment>
-<segment>
-<pinref part="LED5" gate="G$1" pin="VDD"/>
-<pinref part="P+5" gate="1" pin="+5V"/>
-</segment>
-<segment>
-<pinref part="LED6" gate="G$1" pin="VDD"/>
-<pinref part="P+6" gate="1" pin="+5V"/>
-</segment>
-<segment>
-<pinref part="LED7" gate="G$1" pin="VDD"/>
-<pinref part="P+7" gate="1" pin="+5V"/>
-</segment>
-<segment>
-<pinref part="LED8" gate="G$1" pin="VDD"/>
-<pinref part="P+8" gate="1" pin="+5V"/>
-</segment>
 <segment>
 <pinref part="U$2" gate="G$1" pin="1"/>
@@
 <net name="GND" class="0">
 <segment>
-<pinref part="LED8" gate="G$1" pin="GND"/>
-<pinref part="GND1" gate="1" pin="GND"/>
-</segment>
-<segment>
-<pinref part="LED7" gate="G$1" pin="GND"/>
-<pinref part="GND2" gate="1" pin="GND"/>
-</segment>
-<segment>
-<pinref part="LED6" gate="G$1" pin="GND"/>
-<pinref part="GND3" gate="1" pin="GND"/>
-</segment>
-<segment>
-<pinref part="LED5" gate="G$1" pin="GND"/>
-<pinref part="GND4" gate="1" pin="GND"/>
-</segment>
-<segment>
-<pinref part="LED4" gate="G$1" pin="GND"/>
-<pinref part="GND5" gate="1" pin="GND"/>
-</segment>
-<segment>
-<pinref part="LED3" gate="G$1" pin="GND"/>
-<pinref part="GND6" gate="1" pin="GND"/>
-</segment>
-<segment>
-<pinref part="LED2" gate="G$1" pin="GND"/>
-<pinref part="GND7" gate="1" pin="GND"/>
-</segment>
-<segment>
-<pinref part="LED1" gate="G$1" pin="GND"/>
-<pinref part="GND8" gate="1" pin="GND"/>
-</segment>
-<segment>
 <pinref part="U$2" gate="G$1" pin="2"/>
 <wire x1="248.92" y1="-2.54" x2="256.54" y2="-2.54" width="0.1524" layer="91"/>
@@
 <net name="N$8" class="0">
 <segment>
-<pinref part="LED1" gate="G$1" pin="DI"/>
 <wire x1="284.48" y1="-25.4" x2="264.16" y2="-25.4" width="0.1524" layer="91"/>
 <wire x1="264.16" y1="-25.4" x2="264.16" y2="-5.08" width="0.1524" layer="91"/>
@@
 </schematic>
 </drawing>
-<compatibility>
-<note version="8.2" severity="warning">
-Since Version 8.2, EAGLE supports online libraries. The ids
-of those online libraries will not be understood (or retained)
-with this version.
-</note>
-</compatibility>
 </eagle>
