File: nixie_drive/board.sch (EAGLE design)
At the start: 53 parts, among them IC1 74141N, IC2 74HC138D, IC3 74HC138D, U1 ATMEGA328P-AU

Commit message: [fix] 太さ・ガーバー出力(FusionPCB)
Connections:
- net NIXIE1: now also IC1A.1
- net NIXIE2: no longer IC1A.1
Changed lines of the file:
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@@
 <?xml version="1.0" encoding="utf-8"?>
 <!DOCTYPE eagle SYSTEM "eagle.dtd">
-<eagle version="8.4.3">
+<eagle version="8.5.2">
 <drawing>
 <settings>
@@
 <setting verticaltext="up"/>
 </settings>
-<grid distance="0.1" unitdist="inch" unit="inch" style="lines" multiple="1" display="yes" altdistance="0.01" altunitdist="inch" altunit="inch"/>
+<grid distance="0.1" unitdist="inch" unit="inch" style="lines" multiple="1" display="no" altdistance="0.01" altunitdist="inch" altunit="inch"/>
 <layers>
 <layer number="1" name="Top" color="4" fill="1" visible="no" active="no"/>
@@
 </variantdefs>
 <classes>
-<class number="0" name="default" width="0.254" drill="0">
+<class number="0" name="default" width="0.381" drill="0">
+<clearance class="0" value="0.127"/>
 </class>
 </classes>
@@
 </segment>
 <segment>
-<pinref part="IC1" gate="A" pin="1"/>
-<wire x1="134.62" y1="-15.24" x2="139.7" y2="-15.24" width="0.1524" layer="91"/>
-</segment>
-<segment>
 <pinref part="U$4" gate="G$1" pin="P$5"/>
 <wire x1="284.48" y1="111.76" x2="284.48" y2="114.3" width="0.1524" layer="91"/>
@@
 <wire x1="342.9" y1="48.26" x2="342.9" y2="50.8" width="0.1524" layer="91"/>
 </segment>
-</net>
+<segment>
+<pinref part="IC1" gate="A" pin="1"/>
+<wire x1="134.62" y1="-15.24" x2="139.7" y2="-15.24" width="0.1524" layer="91"/>
+</segment>
+</net>
