File: circuit/nixie/vfd_drive.brd (EAGLE design)
At the start: 100 x 100 mm, 51 parts, among them J1 ZX62R-AB-5P, J2 DC_JACK_2DC0005D100, J3 FSM-21045-10, J4 FSM-21045-10, J5 PSM-210223-10, J6 PSM-210223-10, Q1 FA-238V, SW1 SKRPACE010, SW2 SKRPACE010, U1 PIC18F14K50-I, U2 MAX6921AWI+, U3 NJW4131, U4 DS3231M, U5 ADP3338AKCZ-3.3, U9 BME280

Commit message: [update]use backup
Parts:
- moved R21 49.5 mm to (27.7, 62.3), turned to 270 degrees
- moved C19 28.7 mm to (18.3, 60.3), turned to 90 degrees
- moved U9 27.4 mm to (23.6, 60.3), turned to 270 degrees
- moved C18 26.5 mm to (21.1, 60.3), turned to 90 degrees
- moved C2 24.8 mm to (36.5, 72.5), turned to 90 degrees
- moved C3 22.4 mm to (20.4, 74.1), turned to 180 degrees
- moved C4 21.2 mm to (20.4, 71.9), turned to 180 degrees
- moved Q1 12.3 mm to (24.3, 72.9), turned to 270 degrees
- moved SW1 7.00 mm to (11.5, 73.5)
- moved R20 6.55 mm to (29.8, 62.3), turned to 270 degrees
- moved C22 5.38 mm to (16.5, 66.2)
- moved U4 4.13 mm to (21.0, 66.5), turned to 270 degrees
- moved SW2 4.00 mm to (11.5, 67.9)
- moved U1 1.34 mm to (31.0, 70.7)
Connections:
- net D_M renamed D_N
- net +3V3: now also U1.1
- net +5V: no longer U1.1
Routing:
- net GND: track 113.1 -> 181.4 mm
- net +3V3: track 6.30 -> 36.2 mm, vias 0 -> 2
- net SCL: track 0.00 -> 23.1 mm, vias 0 -> 3
- net SDA: track 0.00 -> 21.0 mm, vias 0 -> 2
- net D_P: track 0.00 -> 13.6 mm
- net D_N: track 0.00 -> 12.8 mm
- net N$45: track 0.00 -> 8.92 mm
- net N$44: track 0.00 -> 7.15 mm
- net N$39: track 0.00 -> 1.83 mm
