File: circuit/nixie/vfd_drive.sch (EAGLE design)
At the start: 51 parts, among them J1 ZX62R-AB-5P, J2 DC_JACK_2DC0005D100, J3 FSM-21045-10, J4 FSM-21045-10, J5 PSM-210223-10, J6 PSM-210223-10, Q1 FA-238V, SW1 SKRPACE010, SW2 SKRPACE010, U1 PIC18F14K50-I, U2 MAX6921AWI+, U3 NJW4131, U4 DS3231M, U5 ADP3338AKCZ-3.3, U9 BME280

Commit message: [update]use backup
Connections:
- net D_M renamed D_N
- net +3V3: now also U1.VDD
- net +5V: no longer U1.VDD
Changed lines of the file:
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@@
 <part name="J5" library="taki-library" deviceset="PSM-210223-10" device=""/>
 <part name="J6" library="taki-library" deviceset="PSM-210223-10" device=""/>
-<part name="P+1" library="taki-library" deviceset="+5V" device=""/>
 <part name="SUPPLY7" library="taki-library" deviceset="GND" device=""/>
 <part name="C2" library="taki-library" deviceset="C-EU" device="C0603" value="0.1uF"/>
@@
 <part name="+3V1" library="taki-library" deviceset="+3V3" device=""/>
 <part name="SUPPLY5" library="taki-library" deviceset="GND" device=""/>
+<part name="+3V2" library="180118 Library by matsu" deviceset="+3V3" device=""/>
 </parts>
 <sheets>
@@
 <attribute name="NAME" x="89.535" y="-203.962" size="1.778" layer="95" rot="R180"/>
 </instance>
-<instance part="P+1" gate="1" x="-12.7" y="71.12" smashed="yes">
-<attribute name="VALUE" x="-15.24" y="66.04" size="1.778" layer="96" rot="R90"/>
-</instance>
 <instance part="SUPPLY7" gate="GND" x="48.26" y="55.88" smashed="yes">
 <attribute name="VALUE" x="46.355" y="52.705" size="1.778" layer="96"/>
@@
 <instance part="SUPPLY5" gate="GND" x="-25.4" y="-30.48" smashed="yes">
 <attribute name="VALUE" x="-27.305" y="-33.655" size="1.778" layer="96"/>
+</instance>
+<instance part="+3V2" gate="G$1" x="-12.7" y="71.12" smashed="yes">
+<attribute name="VALUE" x="-15.24" y="66.04" size="1.778" layer="96" rot="R90"/>
 </instance>
 </instances>
@@
 <wire x1="-2.54" y1="-12.7" x2="-2.54" y2="-7.62" width="0.1524" layer="91"/>
 </segment>
+<segment>
+<wire x1="-12.7" y1="68.58" x2="-12.7" y2="66.04" width="0.1524" layer="91"/>
+<pinref part="U1" gate="G$1" pin="VDD"/>
+<wire x1="-12.7" y1="66.04" x2="-10.16" y2="66.04" width="0.1524" layer="91"/>
+<pinref part="+3V2" gate="G$1" pin="+3V3"/>
+</segment>
 </net>
 <net name="EN" class="0">
@@
 </net>
 <net name="+5V" class="0">
-<segment>
-<pinref part="P+1" gate="1" pin="+5V"/>
-<wire x1="-12.7" y1="68.58" x2="-12.7" y2="66.04" width="0.1524" layer="91"/>
-<pinref part="U1" gate="G$1" pin="VDD"/>
-<wire x1="-12.7" y1="66.04" x2="-10.16" y2="66.04" width="0.1524" layer="91"/>
-</segment>
 <segment>
 <pinref part="P+5" gate="1" pin="+5V"/>
@@
 </segment>
 </net>
-<net name="D_M" class="2">
+<net name="D_N" class="2">
 <segment>
 <pinref part="J1" gate="G$1" pin="D-"/>
