File: circuit/nixie/nixie_drive.brd (EAGLE design)
At the start: 200 x 40 mm, 129 parts, among them J1 ZX62R-AB-5P, J2 2DC-0415D200, J3 FSM-21045-20, Q1 2SA1162, Q2 MMSS8050-L, Q3 MMSS8050-L, Q4 TK7P50D, SW1 SKRPACE010, SW2 SKRPACE010, SW3 SKHHLPA010, SW4 SKHHLPA010, SW5 SKHHLPA010, U1 FT231XS, U10 TLP188, U11 TLP188, U12 TLP188, U13 TLP188, U14 TLP188, U15 TLP188, U16 TLP188, U17 TLP188, U18 GYSFDMAXB, U19 74HC595D, U2 ESP-WROOM-32, U20 MP2307, U3 NJM2360AM, U4 DS3231M, U5 SN75468, U6 74HC595D, U7 SN75468, U8 74HC138D, U9 BME280

Commit message: update nixie
Parts:
- added R41, R9: 4.7k, taki-library:R0603
Connections:
- removed net N$37: R32.2, U18.6
- new net 1PPS: R32.2, U18.6, U2.10
- new net 32KHZ: R41.1, U2.37, U4.1
- new net SQW: R9.1, U2.6, U4.3
- net +3V3: now also R41.2, R9.2
Routing:
- net 1PPS: track 0.00 -> 57.3 mm, vias 0 -> 5
- net 32KHZ: track 0.00 -> 40.0 mm, vias 0 -> 4
- net SQW: track 0.00 -> 33.2 mm, vias 0 -> 4
- net N$37: track 15.1 -> 0.00 mm, vias 2 -> 0
- net +3V3: track 332.8 -> 337.0 mm
- net GND1: track 45.4 -> 41.4 mm
- net GND: track 693.4 -> 695.8 mm, vias 176 -> 174
- net SCL: track 46.7 -> 47.8 mm
- net TXD: track 77.0 -> 77.5 mm
