File: circuit/nixie/nixie_drive.brd (EAGLE design)
At the start: 200 x 40 mm, 136 parts, among them J1 ZX62R-AB-5P, J2 2DC-0415D200, J3 FSM-21045-20, Q1 2SA1162, Q2 MMSS8050-L, Q3 MMSS8050-L, Q4 TK7P50D, Q5 FA-238V, SW1 SKRPACE010, SW2 SKRPACE010, SW3 SKHHLPA010, SW4 SKHHLPA010, SW5 SKHHLPA010, SW6 SKRPACE010, U1 FT231XS, U10 TLP188, U11 TLP188, U12 TLP188, U13 TLP188, U14 TLP188, U15 TLP188, U16 TLP188, U17 TLP188, U18 ATMEGA328P-AU-TQFP32, U19 74HC595D, U2 ESP-WROOM-32, U20 MP2307, U3 NJM2360AM, U4 DS3231M, U5 SN75468, U6 74HC595D, U7 SN75468, U9 BME280

Commit message: [temp]破壊的変更前の
Parts:
- removed C36: (no value), taki-library:C5750
- removed D2: S2MS2M, taki-library:MKT-DO214AA
- removed VR1: SM-42A, taki-library:SM-42A
- added R33: 10k, taki-library:R0603
- added R57: 2.4k, taki-library:R0603
- added U8: MCP4017, taki-library:SC-70-MICROCHIP
- C1: value UWT1E221MNL1GS -> 10uF; device taki-library:NICHICON-ALMINUM-CAPACITOR-8MM -> taki-library:C0603
- C12: value 1500pF -> 0.1uF
- C3: value 0.1uF -> 10uF
- C9: value ULR2D330MML1GS -> 10nF; device taki-library:NICHICON-ALMINUM-CAPACITOR-10MM -> taki-library:C0603
- D1: value 1SS400SM -> RFN2L4STE25; device taki-library:EMD2 -> taki-library:SOD-106
- L1: value CLF12577NIT-221M-D -> LPR6235; device taki-library:CLF12577NI-D -> taki-library:LPR6235
- Q1: value 2SA1162 -> IRLML6344TRPBFTR; device taki-library:SOT346 -> taki-library:SOT23-N-MOSFET
- Q4: value TK7P50D -> IRLML6344TRPBFTR; device taki-library:2-7K1A -> taki-library:SOT23-N-MOSFET
- R11: value 330k -> 0.1
- R12: value 470 -> 1k
- R13: value 1k -> 20
- R14: value 2k -> 174k
- R44: value 0.25 -> 1k; device taki-library:R5025 -> taki-library:R0603
- R45: value 1k -> 360k
- U3: value NJM2360AM -> LM3478; device taki-library:DMP8 -> taki-library:SOIC8-LT
- moved C34 232.5 mm to (195.0, 30.0)
- moved R45 230.8 mm to (-13.0, -105.0), turned to 0 degrees
- moved Q4 219.7 mm to (-11.0, -84.0), turned to 0 degrees
- moved C35 219.1 mm to (178.0, 29.0), turned to 90 degrees
- moved C9 217.4 mm to (-13.0, -41.0), turned to 0 degrees
- moved R14 215.8 mm to (-13.0, -71.0)
- moved R11 211.3 mm to (-13.0, -35.0), turned to 0 degrees
- moved C12 205.1 mm to (-13.0, -59.0), turned to 0 degrees
- moved R44 203.1 mm to (-13.0, -91.0), turned to 0 degrees
- moved R13 202.1 mm to (-13.0, -65.0), turned to 0 degrees
- moved C11 196.0 mm to (-13.0, -47.0), turned to 0 degrees
- moved C33 193.8 mm to (167.0, 5.00)
- moved R31 193.8 mm to (167.0, 11.0)
- moved R32 193.8 mm to (172.0, 11.0)
- moved R12 192.0 mm to (-13.0, -53.0), turned to 0 degrees
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Connections:
- net GND1 renamed N$50
- removed net 1PPS: U2.10
- removed net N$81: L1.1, R12.2, R13.2, R44.2, U3.7
- new net FB: R57.2, U3.3, U8.5
- new net GPS_RX: U2.28
- new net GPS_TX: U2.27
- new net N$39: Q4.G, R44.2
- new net N$49: R45.1, U8.6
- new net SCL_AT: U18.28, U8.3
- new net SDA_AT: U18.27, U8.4
- new net UC_EN: R44.1, U18.17
- net +12V: now also C1.1, L1.1, R13.1, R33.2; no longer C1.POS, R44.1, U3.6
- net +200V: now also C34.1, C35.1, D1.K, R45.2; no longer C9.POS, D2.K, R11.2
- net +3V3: now also U8.1
- net GND: now also C1.2, C34.2, C35.2, C9.2, R11.1, R12.1, R57.1, U3.5, U8.2; no longer C1.NEG, C11.2, C9.NEG, Q1.3, R14.1, R45.1
- net N$14: now also L1.2, L1.4, Q1.D; no longer D1.K, Q1.2, Q4.G
- net N$15: now also C11.1; no longer D1.A, Q1.1, R45.2
- net N$16: now also R14.2, U3.7; no longer D2.A, L1.2, Q4.D
- net N$18: now also D1.A, L1.3; no longer R11.1, VR1.1
- net N$19: now also Q1.G, U3.6; no longer R12.1, U3.8
- net N$20: now also C9.1, Q1.S, R11.2; no longer R13.1
- net N$21: now also C11.2, R12.2; no longer R14.2, VR1.3
- net N$23: now also C12.1, R13.2, U3.8; no longer C11.1, U3.5, VR1.2
- net N$24: now also Q4.D, R14.1, R33.1; no longer C12.1, U3.3
Routing:
- net +200V: track 144.9 -> 62.3 mm, vias 2 -> 0
- net GND: track 627.7 -> 569.2 mm, vias 127 -> 103
- net N$50: track 41.4 -> 0.00 mm, vias 6 -> 0
- net N$81: track 35.1 -> 0.00 mm
- net +12V: track 212.5 -> 177.5 mm
- net N$23: track 22.8 -> 0.00 mm, vias 2 -> 0
- net N$16: track 17.5 -> 0.00 mm
- net N$14: track 17.0 -> 0.00 mm, vias 2 -> 0
- net N$15: track 11.1 -> 0.00 mm
- net N$24: track 8.88 -> 0.00 mm
- net N$21: track 8.28 -> 0.00 mm
- net N$20: track 3.87 -> 0.00 mm
- net N$19: track 3.49 -> 0.00 mm
- net N$18: track 3.45 -> 0.00 mm
- net 1PPS: track 1.50 -> 0.00 mm, vias 1 -> 0
- removed copper zone on layer 1, net N$85
- removed copper zone on layer 16, net N$85

Commit message: [add]add all:wq
Parts:
- removed C27: 10nF, taki-library:C0603
- removed D4: B130LAW-7-F, taki-library:DIODE-ZETEX-SOD123
- removed L2: NR10050T100M, taki-library:NR10050T100M
- removed R53: 100k, taki-library:R0603
- removed R54: 26.1k/1%, taki-library:R0603
- removed R55: 10k/1%, taki-library:R0603
- removed R56: 6.8k, taki-library:R0603
- added J4: PIN_HEADER_MALE_1X05_05P, taki-library:PIN_HEADER_MALE_1X05_05P
- added J5: ZX62R-AB-5P, taki-library:ZX62R-B-5PA
- added SP1: PKLCS1212E4001-R1, taki-library:PKLCS1212E4001-R1
- added U22: FT232RL, taki-library:SSOP28
- C24: value 10uF -> 10nF
- C26: value 0.1uF -> 10uF
- C28: value 3.9nF -> 0.1uF
- C29: value 22μF -> UWT1E221MNL1GS; device taki-library:C2012 -> taki-library:NICHICON-ALMINUM-CAPACITOR-8MM
- C30: value 22μF -> 0.1u; device taki-library:C2012 -> taki-library:C0603
- C33: value 1000pF -> 0.1uF
- J2: value 2DC-0415D200 -> DC_JACK_2DC0005D100; device taki-library:2DC-0415D200 -> taki-library:DC_JACK_2DC0005D100
- R32: value 470 -> 1k
- R41: value 4.7k -> 0
- U20: value MP2307 -> ADP3338AKCZ-3.3; device taki-library:MP2307 -> taki-library:SOT233
- moved R45 235.7 mm to (193.9, 7.94)
- moved R57 225.3 mm to (177.1, 9.88)
- moved U8 221.5 mm to (180.1, 12.2), turned to 180 degrees
- moved R13 210.3 mm to (176.3, 26.6), turned to 270 degrees
- moved R44 207.8 mm to (168.7, 9.76), turned to 90 degrees
- moved R14 206.2 mm to (173.7, 16.4)
- moved R33 206.0 mm to (170.6, 16.4), turned to 180 degrees
- moved Q4 206.0 mm to (171.4, 11.6)
- moved C12 205.9 mm to (175.4, 24.0), turned to 180 degrees
- moved C3 203.7 mm to (181.0, 33.0), turned to 90 degrees
- moved R11 201.7 mm to (182.0, 16.8), turned to 90 degrees
- moved C1 199.0 mm to (178.0, 33.0), turned to 90 degrees
- moved C11 193.0 mm to (168.0, 20.0), turned to 180 degrees
- moved C9 192.8 mm to (168.9, 23.1), turned to 90 degrees
- moved R12 192.3 mm to (164.9, 20.0)
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Connections:
- removed net +12V: C1.1, C24.1, C25.1, C3.1, J2.1, L1.1, R13.1, R33.2, R53.1, U20.2
- removed net 32KHZ: R41.1, U2.37, U4.1
- removed net N$88: R53.2, U20.7
- removed net N$89: C26.1, U20.8
- removed net N$91: R54.1, R55.2, U20.5
- removed net N$92: C27.2, U20.1
- removed net N$93: C27.1, D4.K, L2.P$1, U20.3
- removed net N$95: C28.1, U20.6
- removed net N$96: C28.2, R56.2
- new net +5V: C1.1, C26.1, C29.POS, C3.1, J2.1, L1.1, R13.1, R33.2, U20.3
- new net N$76: R41.2, R45.1
- new net N$77: C30.1, J4.P$2
- new net N$78: C33.1, U22.17
- new net N$81: C2.1, C23.1, U18.18, U18.4, U18.6
- new net N$82: J5.D+, U22.15
- new net N$83: J5.D-, U22.16
- new net SPEAKER: R32.2, U2.26
- net +3V3: now also C25.1, C28.1, J4.P$1, U20.2, U20.4, U22.20, U22.4; no longer C2.1, C23.1, C29.1, C30.1, L2.P$2, R41.2, R54.2, U18.18, U18.4, U18.6
- net ESP32_RX: now also J4.P$4, U2.27; no longer U2.24
- net ESP32_TX: now also J4.P$3, U2.28; no longer U2.23
- net FB: now also C24.1
- net GND: now also C28.2, C29.NEG, C33.2, J4.P$5, SP1.2, U20.1, U22.18, U22.21, U22.25, U22.26, U22.7; no longer C29.2, C30.2, C33.1, D4.A, R55.1, R56.1, U20.4, U20.PAD
- net GPS_RX: now also U2.23; no longer U2.28
- net GPS_TX: now also U2.24; no longer U2.27
- net N$37: now also SP1.1; no longer C33.2, SW6.S1, SW6.S2
- net N$49: now also R41.1; no longer R45.1
- net RST: now also C30.2, SW6.S1, SW6.S2; no longer R32.2
Routing:
- net +12V: track 177.5 -> 0.00 mm, vias 2 -> 0
- net GND: track 569.2 -> 695.0 mm, vias 103 -> 241
- net +3V3: track 301.3 -> 415.1 mm, vias 8 -> 16
- net SCL_AT: track 0.00 -> 110.7 mm, vias 0 -> 4
- net SDA_AT: track 0.00 -> 109.3 mm, vias 0 -> 4
- net UC_EN: track 0.00 -> 94.5 mm, vias 0 -> 2
- net +200V: track 62.3 -> 151.7 mm
- net N$64: track 7.20 -> 75.2 mm, vias 1 -> 2
- net +5V: track 0.00 -> 58.3 mm
- net N$50: track 0.00 -> 43.6 mm, vias 0 -> 6
- net SCL: track 30.5 -> 71.4 mm, vias 2 -> 5
- net SDA: track 27.0 -> 67.2 mm, vias 2 -> 3
- net RST: track 0.00 -> 28.3 mm
- net FB: track 0.00 -> 22.5 mm, vias 0 -> 2
- net SQW: track 0.22 -> 20.7 mm, vias 0 -> 2
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Other:
- outline, holes or cut-outs redrawn
- board text added: "nixie tube drive board rev.3"
- board text removed: "NIT,Tokyo College meister2018"
- board text removed: "nixie tube drive board rev.2"
