File: circuit/nixie/nixie_drive.sch (EAGLE design)
At the start: 129 parts, among them J1 ZX62R-AB-5P, J2 2DC-0415D200, J3 FSM-21045-20, Q1 2SA1162, Q2 MMSS8050-L, Q3 MMSS8050-L, Q4 TK7P50D, SW1 SKRPACE010, SW2 SKRPACE010, SW3 SKHHLPA010, SW4 SKHHLPA010, SW5 SKHHLPA010, U1 FT231XS, U10 TLP188, U11 TLP188, U12 TLP188, U13 TLP188, U14 TLP188, U15 TLP188, U16 TLP188, U17 TLP188, U18 GYSFDMAXB, U19 74HC595D, U2 ESP-WROOM-32, U20 MP2307, U3 NJM2360AM, U4 DS3231M, U5 SN75468, U6 74HC595D, U7 SN75468, U8 74HC138D, U9 BME280

Commit message: update nixie
Parts:
- added R41, R9: 4.7k, taki-library:R-EU_R0603
Connections:
- removed net N$37: R32.2, U18.IPPS
- new net 1PPS: R32.2, U18.IPPS, U2.IO25
- new net 32KHZ: R41.1, U2.IO23, U4.32KHZ
- new net SQW: R9.1, U2.IO34, U4.SQW
- net +3V3: now also R41.2, R9.2
Other:
- moved on the sheet: C18, C19, C22, R20, R21, U9
