File: circuit/nixie/nixie_drive.sch (EAGLE design)
At the start: 136 parts, among them J1 ZX62R-AB-5P, J2 2DC-0415D200, J3 FSM-21045-20, Q1 IRLML6344TRPBFTR, Q2 MMSS8050-L, Q3 MMSS8050-L, Q4 IRLML6344TRPBFTR, Q5 FA-238V, SW1 SKRPACE010, SW2 SKRPACE010, SW3 SKHHLPA010, SW4 SKHHLPA010, SW5 SKHHLPA010, SW6 SKRPACE010, U1 FT231XS, U10 TLP188, U11 TLP188, U12 TLP188, U13 TLP188, U14 TLP188, U15 TLP188, U16 TLP188, U17 TLP188, U18 ATMEGA328P-AU-TQFP32, U19 74HC595D, U2 ESP-WROOM-32, U20 MP2307, U3 LM3478, U4 DS3231M, U5 SN75468, U6 74HC595D, U7 SN75468, U8 MCP4017, U9 BME280

Commit message: [add]add all:wq
Parts:
- removed C27: 10nF, taki-library:C-EUC0603
- removed D4: B130LAW-7-F, taki-library:B130LAW-7-F
- removed L2: NR10050T100M, taki-library:NR10050T100M
- removed R53: 100k, taki-library:R-EU_R0603
- removed R54: 26.1k/1%, taki-library:R-EU_R0603
- removed R55: 10k/1%, taki-library:R-EU_R0603
- removed R56: 6.8k, taki-library:R-EU_R0603
- added J4: PIN_HEADER_MALE_1X05_05P, taki-library:PIN_HEADER_MALE_1X05_05P
- added J5: ZX62R-AB-5P, taki-library:ZX62R-AB-5P
- added SP1: PKLCS1212E4001-R1, taki-library:PKLCS1212E4001-R1
- added U22: FT232RL, taki-library:FT232RL
- C24: value 10uF -> 10nF
- C26: value 0.1uF -> 10uF
- C28: value 3.9nF -> 0.1uF
- C29: value 22μF -> UWT1E221MNL1GS; device taki-library:C-EUC2012 -> taki-library:UWT1E221MNL1GS
- C30: value 22μF -> 0.1u; device taki-library:C-EUC2012 -> taki-library:C-EUC0603
- C33: value 1000pF -> 0.1uF
- J2: value 2DC-0415D200 -> DC_JACK_2DC0005D100; device taki-library:2DC-0415D200 -> taki-library:DC_JACK_2DC0005D100
- R32: value 470 -> 1k
- R41: value 4.7k -> 0
- U20: value MP2307 -> ADP3338AKCZ-3.3; device taki-library:MP2307 -> taki-library:ADP3338AKCZ-3.3
Connections:
- removed net +12V: C1.1, C24.1, C25.1, C3.1, J2.1, L1.1, R13.1, R33.2, R53.1, U20.IN
- removed net 32KHZ: R41.1, U2.IO23, U4.32KHZ
- removed net N$88: R53.2, U20.EN
- removed net N$89: C26.1, U20.SS
- removed net N$91: R54.1, R55.2, U20.FB
- removed net N$92: C27.2, U20.BS
- removed net N$93: C27.1, D4.C, L2.1, U20.SW
- removed net N$95: C28.1, U20.COMP
- removed net N$96: C28.2, R56.2
- new net +5V: C1.1, C26.1, C29.+, C3.1, J2.1, L1.1, R13.1, R33.2, U20.IN
- new net N$76: R41.2, R45.1
- new net N$77: C30.1, J4.2
- new net N$78: C33.1, U22.3V3OUT
- new net N$81: C2.1, C23.1, U18.AVCC, U18.VCC@1, U18.VCC@2
- new net N$82: J5.D+, U22.USBDP
- new net N$83: J5.D-, U22.USBDM
- new net SPEAKER: R32.2, U2.IO4
- net +3V3: now also C25.1, C28.1, J4.1, U20.OUT, U22.VCC, U22.VCCIO; no longer C2.1, C23.1, C29.1, C30.1, L2.2, R41.2, R54.2, U18.AVCC, U18.VCC@1, U18.VCC@2
- net ESP32_RX: now also J4.4, U2.IO16; no longer U2.IO2
- net ESP32_TX: now also J4.3, U2.IO17; no longer U2.IO15
- net FB: now also C24.1
- net GND: now also C28.2, C29.-, C33.2, J4.5, SP1.P$2, U22.GND, U22.GND@1, U22.GND@2, U22.GND@A, U22.TEST; no longer C29.2, C30.2, C33.1, D4.A, R55.1, R56.1
- net GPS_RX: now also U2.IO15; no longer U2.IO17
- net GPS_TX: now also U2.IO2; no longer U2.IO16
- net N$37: now also SP1.1; no longer C33.2, SW6.S, SW6.S1
- net N$49: now also R41.1; no longer R45.1
- net RST: now also C30.2, SW6.S, SW6.S1; no longer R32.2
Other:
- moved on the sheet: BATT1, C10, C13, C14, C17, C18, C19, C20, C21, C22, C24, C25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

Commit message: [update]
Parts:
- removed LED3: VBUS, taki-library:LEDCHIPLED_0603
- removed R10: 1k, taki-library:R-EU_R0603
- removed R15: 4.7k, taki-library:R-EU_R0603
- removed R16: 10k, taki-library:R-EU_R0603
- removed R17, R18: 27, taki-library:R-EU_R0603
- removed U1: FT231XS, taki-library:FT231XS
- added C27: 0.1u, taki-library:C-EUC0603
- added C36, C37: (no value), taki-library:C-EUC0603
- added U21: FT232RL, taki-library:FT232RL
- C13, C14: value 47pF -> 0.1uF
- C29: value UWT1E221MNL1GS -> (none); device taki-library:UWT1E221MNL1GS -> taki-library:C-EUC0603
- R31: value 10k -> 1k
Connections:
- net N$83 renamed D2_M
- removed net D2_N: R17.2, U1.USBDM
- removed net D_N: C13.1, J1.D-, R17.1
- removed net D_P: C14.1, J1.D+, R18.1
- removed net ESP32_RX: J4.4, U18.PD1(TXD), U2.IO16
- removed net ESP32_TX: J4.3, U18.PD0(RXD), U2.IO17
- removed net GPS_RX: U2.IO15
- removed net GPS_TX: U2.IO2
- removed net N$81: C2.1, C23.1, U18.AVCC, U18.VCC@1, U18.VCC@2
- removed net N$82: J5.D+, U22.USBDP
- removed net VBUS: J1.VBUS, R10.2, R15.2
- new net AVR_RX: J4.4, U18.PD0(RXD), U2.IO2, U22.TXD
- new net AVR_TX: J4.3, U18.PD1(TXD), U2.IO15, U22.RXD
- new net D1_M: J1.D-, U21.USBDM
- new net D1_P: J1.D+, U21.USBDP
- new net N$84: C13.1, U21.3V3OUT, U21.VCCIO
- new net N$85: C4.1, J1.VBUS, U21.VCC
- net +3V3: now also C2.1, C23.1, U18.AVCC, U18.VCC@1, U18.VCC@2; no longer C4.1, U1.!RESET, U1.3V3OUT, U1.VCC, U1.VCCIO, U22.VCC, U22.VCCIO
- net +5V: now also C29.1, C36.1, C37.1; no longer C29.+
- net D2_P: now also J5.D+, U22.USBDP; no longer R18.2, U1.USBDP
- net DTR: now also U21.!DTR; no longer U1.!DTR
- net GND: now also C29.2, C36.2, C37.2, J5.GND, J5.SHIELD, U21.GND, U21.GND@1, U21.GND@2, U21.GND@A, U21.TEST; no longer C29.-, LED3.C, R16.1, U1.GND@16, U1.GND@6
- net N$13: now also C14.1, J5.VBUS, U22.VCC; no longer LED3.A, R10.1
- net N$2: now also C27.1, U22.!RTS; no longer R15.1, R16.2, U1.CBUS0
- net N$4: now also U21.CBUS1; no longer U1.CBUS1
- net N$5: now also U21.CBUS0; no longer U1.CBUS2
- net N$78: now also U22.VCCIO
- net RST: now also C27.2
- net RTS: now also U21.!RTS; no longer U1.!RTS
- net RXD: now also U21.RXD; no longer U1.RXD
- net TXD: now also U21.TXD; no longer U1.TXD
Other:
- moved on the sheet: BATT1, C13, C14, C18, C19, C22, C30, C4, J1, J4, LED1, LED2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
