File: circuit/nixie/nixie_drive_neo.sch (EAGLE design)
At the start: 75 parts, among them J1 ZX62R-AB-5P, J2 2DC-0415D200, J3 FSM-21045-7, J4 PSM-210223-7, J5 PSM-210223-7, J6 FSM-21045-7, Q1 BSS138, Q2 BSS138, SW1 SKRPACE010, SW2 SKRPACE010, SW3 JTP1230D, SW4 JTP1230D, SW5 JTP1230D, SW6 JTP1230D, U1 FT231XS, U2 MAX6921AWI+, U3 NJW4131, U4 DS3231M, U5 ADP3338AKCZ-3.3, U6 PSF-A85, U9 BME280

Commit message: [add]add all
Parts:
- removed C24: 1000pF, taki-library:C-EUC0603
- removed D2: BZX584C3V9, taki-library:BZX584C3V9
- removed DIS1: IV18, taki-library:IV18
- removed J2: 2DC-0415D200, taki-library:2DC-0415D200
- removed J6: FSM-21045-7, taki-library:FSM-21045-7
- removed R10: 4.7k, taki-library:R-EU_R0603
- removed R15: 10k, taki-library:R-EU_R0603
- removed R17, R18: 27, taki-library:R-EU_R0603
- removed U1: FT231XS, taki-library:FT231XS
- removed VR1: PVZ3A104C01, taki-library:PVZ3A104C01
- added C27, C30: 0.1u, taki-library:C-EUC0603
- added C31, C32: 33p, taki-library:C-EUC0603
- added C33: 0.1uF, taki-library:C-EUC0603
- added C34, C35: 1u, taki-library:C-EU
- added D3: MMSZ5267BT1G, taki-library:MMSZ5267BT1G
- added LED6: LED1, taki-library:LEDCHIPLED_0603
- added Q3: MMSS8050-L, taki-library:MMSS8050-L
- added Q4: IRLML6344TRPBFTR, taki-library:IRLML6344TRPBFTR
- added Q5: FA-238V, taki-library:FA-238V
- added R19: 220k, taki-library:R-EU_R0603
- added R22, R26, R27, R28, R29: 10k, taki-library:R-EU_R3216
- added R30, R34, R35, R36, R37, R38, R39, R40, R42, R43: 1k, 180118 Library by matsu:R-EU_R0603
- added R31, R32, R44, R46: 1k, taki-library:R-EU_R0603
- added R33, R48, R50, R52: 10k, taki-library:R-EU_R0603
- added R41: 0, taki-library:R-EU_R0603
- added R45: 360k, taki-library:R-EU_R0603
- added R47, R49, R51: 470, taki-library:R-EU_R0603
- added R57: 2.4k, taki-library:R-EU_R0603
- added SP1: PKLCS1212E4001-R1, taki-library:PKLCS1212E4001-R1
- added U10, U11, U12, U13, U14, U15, U16, U17: TLP188, taki-library:TLP188
- added U18: ATMEGA328P-AU-TQFP32, taki-library:MCU-ATMEGA328P-AU(TQFP32)
- added U19: 74HC595D, taki-library:74HC595D
- added U21, U22: FT232RL, taki-library:FT232RL
- added U7: SN75468, taki-library:SN75468
- C1: value 0.1uF -> 10uF
- C10: value 0.1uF -> 1000pF
- C11: value 10uF -> 0.1uF; device taki-library:C-EUC3216 -> taki-library:C-EUC0603
- C13: value 10uF -> 0.1uF
- C14: value 270pF -> 0.1uF
- C16: value 47pF -> 0.1uF
- C17: value 47pF -> 1000pF
- C2: value 10uF -> 0.1u; device taki-library:C-EUC3216 -> taki-library:C-EUC0603
- C23: value 1000pF -> 0.1u
- C3: value 1uF -> 10uF
- C4: value 1uF -> 0.1uF
- C5: value (none) -> 0.1uF; device taki-library:C-EUC3225 -> taki-library:C-EUC0603
- C6: value 10uF -> 100uF; device taki-library:C-EUC0603 -> taki-library:C-EUC1210
- C9: value 10uF -> 10nF
- D1: value SS2040FL -> RFN2L4STE25; device taki-library:SS2040FL -> taki-library:RFN2L4STE25
- J3: value FSM-21045-7 -> FSM-21045-20; device taki-library:FSM-21045-7 -> taki-library:FSM-21045-20
- J4: value PSM-210223-7 -> PIN_HEADER_MALE_1X05_05P; device taki-library:PSM-210223-7 -> taki-library:PIN_HEADER_MALE_1X05_05P
- J5: value PSM-210223-7 -> ZX62R-AB-5P; device taki-library:PSM-210223-7 -> taki-library:ZX62R-AB-5P
- L1: value NR10050T470M -> LPR6235; device taki-library:NR10050T470M -> taki-library:LPR6235
- Q1: value BSS138 -> IRLML6344TRPBFTR; device taki-library:BSS138 -> taki-library:IRLML6344TRPBFTR
- Q2: value BSS138 -> MMSS8050-L; device taki-library:BSS138 -> taki-library:MMSS8050-L
- R1: value 27k -> 1k
- R11: value 27k -> 0.1
- R13: value 1k -> 20
- R14: value 10k -> 174k
- R2: value 8.2k -> 1k
- R23, R24: device taki-library:R-EU_R0603 -> taki-library:R-EU_R3216
- R25: value 4.7k -> 10k; device taki-library:R-EU_R0603 -> taki-library:R-EU_R3216
- R4, R6: value 10k -> 470
- R7: value 27k -> 10k
- R8: value 3.3k -> 10k
- R9: value 3.3k -> 4.7k
- SW3, SW4, SW5: value JTP1230D -> SKHHLPA010; device taki-library:JTP1230D -> taki-library:SKHHLPA010
- SW6: value JTP1230D -> SKRPACE010; device taki-library:JTP1230D -> taki-library:SKRPACE010
- U2: value MAX6921AWI+ -> ESP-WROOM-32; device taki-library:MAX6921AWI+ -> taki-library:ESP-WROOM-32
- U3: value NJW4131 -> LM3478; device taki-library:NJW4131 -> taki-library:LM3478
- U5: value ADP3338AKCZ-3.3 -> SN75468; device taki-library:ADP3338AKCZ-3.3 -> taki-library:SN75468
- U6: value PSF-A85 -> 74HC595D; device ITEAD:PSF-A85 -> taki-library:74HC595D
Connections:
- removed net +24V: C11.1, C2.1, D1.C, R7.1, R8.1, U2.VBB
- removed net 32KHZ: R10.1, U4.32KHZ, U6.GPIO12
- removed net D2_N: R17.2, U1.USBDM
- removed net D_N1: C16.1, J1.D-, R17.1
- removed net D_P1: C17.1, J1.D+, R18.1
- removed net N$49: R8.2, VR1.E, VR1.S
- removed net RESET: C8.2, Q1.D, R3.1, SW1.S, SW1.S1, U6.RESET
- removed net SW1: J4.2, U6.GPIO5
- removed net SW1-SW: C20.2, J6.2, R4.1, SW3.S, SW3.S1
- removed net SW2: J4.3, U6.GPIO8
- removed net SW2-SW: C21.2, J6.3, R6.1, SW4.S, SW4.S1
- removed net SW3-SW: C23.2, J6.4, R14.1, SW5.S, SW5.S1
- removed net SW4-SW: C24.2, J6.5, R15.1, SW6.S, SW6.S1
- removed net VBUS: J1.VBUS
- removed net VFBLANK: J3.6, U6.GPIO4
- removed net VFCLK: J3.4, U6.GPIO10
- removed net VFD10: DIS1.B, U2.OUT4
- removed net VFD11: DIS1.F, U2.OUT5
- removed net VFD12: DIS1.A, U2.OUT6
- removed net VFD14: DIS1.9, U2.OUT8
- removed net VFD15: DIS1.1, U2.OUT9
- removed net VFD16: DIS1.3, U2.OUT16
- removed net VFD17: DIS1.5, U2.OUT15
- removed net VFD18: DIS1.8, U2.OUT14
- removed net VFD19: DIS1.7, U2.OUT13
- removed net VFD2: DIS1.H, U2.OUT7
- removed net VFD20: DIS1.6, U2.OUT12
- removed net VFD21: DIS1.4, U2.OUT11
- removed net VFD22: DIS1.2, U2.OUT10
- removed net VFD3: DIS1.D, U2.OUT0
- removed net VFD4: DIS1.C, U2.OUT1
- removed net VFD5: DIS1.E, U2.OUT2
- removed net VFD9: DIS1.G, U2.OUT3
- removed net VFDIN: J3.3, U6.GPIO11
- removed net VFLOAD: J3.5, U6.GPIO9
- new net +200V: C34.1, C35.1, D1.C, R19.2, R45.2, U10.COL, U11.COL, U12.COL, U13.COL, U14.COL, U15.COL, U16.COL, U17.COL
- new net ANODE1: J3.13, R22.2
- new net ANODE2: J3.14, R23.2
- new net ANODE3: J3.15, R24.2
- new net ANODE4: J3.16, R25.2
- new net ANODE5: J3.17, R26.2
- new net ANODE6: J3.18, R27.2
- new net ANODE7: J3.19, R28.2
- new net ANODE8: J3.20, R29.2
- new net AVR_RX: J4.4, U18.PD0(RXD), U2.IO2, U22.TXD
- new net AVR_TX: J4.3, U18.PD1(TXD), U2.IO15, U22.RXD
- new net D1_M: J1.D-, U21.USBDM
- new net D1_P: J1.D+, U21.USBDP
- new net D2_M: J5.D-, U22.USBDM
- new net EN: C7.1, Q2.C, R3.1, R4.2, U2.EN
- new net FB: R41.1, R57.2, U3.FB
- new net N$11: C32.1, Q5.3, U18.PB7(XTAL2/TOSC2)
- new net N$12: C10.2, R6.1, SW2.S, SW2.S1
- new net N$13: C14.1, J5.VBUS, U22.VCC
- new net N$14: L1.2, L1.4, Q1.D
- new net N$15: C11.1, U3.COMP
- new net N$16: R14.2, U3.FA/SD
- new net N$17: U6A.QA, U7.1B
- new net N$20: C9.1, Q1.S, R11.2, U3.ISEN
- new net N$22: U5.7B, U6A.QB
- new net N$23: C12.1, R13.2, U3.VIN
- new net N$24: Q4.D, R14.1, R33.1
- new net N$25: U5.6B, U6A.QC
- new net N$26: U5.5B, U6A.QD
- new net N$27: C31.1, Q5.1, U18.PB6(XTAL1/TOSC1)
- new net N$28: R22.1, U10.EMIT
- new net N$29: R23.1, U11.EMIT
- new net N$30: R24.1, U12.EMIT
- new net N$31: R25.1, U13.EMIT
- new net N$32: R26.1, U14.EMIT
- new net N$33: R27.1, U15.EMIT
- new net N$34: R28.1, U16.EMIT
- new net N$35: R29.1, U17.EMIT
- new net N$36: R30.2, U10.A
- new net N$37: R32.1, SP1.1
- new net N$38: U10.C, U18.PD2(INT0)
- new net N$39: Q4.G, R44.2
- new net N$42: U5.2B, U6A.QG
- new net N$44: U19A.SER, U6A.QH*
- new net N$45: U19A.QA, U7.7B
- new net N$50: LED6.C, U2.IO32
- new net N$51: R34.2, U11.A
- new net N$52: R35.2, U12.A
- new net N$53: R36.2, U13.A
- new net N$54: R37.2, U14.A
- new net N$55: R38.2, U15.A
- new net N$56: R39.2, U16.A
- new net N$57: R40.2, U17.A
- new net N$58: U11.C, U18.PD3(INT1)
- new net N$59: U12.C, U18.PD4(XCK/T0)
- new net N$6: C8.2, R4.1, SW1.S, SW1.S1
- new net N$60: U13.C, U18.PD5(T1)
- new net N$61: U14.C, U18.PD6(AIN0)
- new net N$62: U15.C, U18.PD7(AIN1)
- new net N$63: U16.C, U18.PB0(ICP)
- new net N$64: U17.C, U18.PB1(OC1A)
- new net N$65: J3.2, U5.2C
- new net N$66: J3.3, U5.3C
- new net N$67: J3.4, U5.4C
- new net N$68: J3.5, U5.5C
- new net N$69: J3.6, U5.6C
- new net N$70: J3.7, U5.7C
- new net N$71: J3.8, U7.1C
- new net N$72: J3.9, U7.2C
- new net N$73: J3.10, U7.3C
- new net N$74: J3.11, R42.2
- new net N$75: J3.12, R43.2
- new net N$76: R41.2, R45.1
- new net N$77: C30.1, J4.2
- new net N$78: C33.1, U22.3V3OUT, U22.VCCIO
- new net N$79: R42.1, U7.4C
- new net N$80: R43.1, U7.7C
- new net N$84: C13.1, U21.3V3OUT, U21.VCCIO
- new net N$85: C4.1, J1.VBUS, U21.VCC
- new net N$86: C20.2, R49.1, SW4.2
- new net N$87: C17.2, R47.1, SW3.2
- new net N$90: C21.2, R51.1, SW5.2
- new net N$94: LED6.A, R46.1
- new net RCK: U18.PB4(MISO), U19A.RCK, U6A.RCK
- new net RST: C27.2, C30.2, R31.1, SW6.S, SW6.S1, U18.PC6(/RESET)
- new net SCK: U18.PB3(MOSI/OC2), U19A.SCK, U6A.SCK
- new net SCL_AT: U18.PC5(ADC5/SCL)
- new net SDA_AT: U18.PC4(ADC4/SDA)
- new net SER: U18.PB2(SS/OC1B), U6A.SER
- new net SPEAKER: R32.2, U2.IO4
- new net SW5: R51.2, R52.1, U2.IO14
- new net UC_EN: R44.1, U18.PB5(SCK)
- net +3V3: now also C16.1, C2.1, C23.1, C5.1, C6.1, R1.2, R2.2, R30.1, R31.2, R34.1, R35.1, R36.1, R37.1, R38.1, R39.1, R40.1, R46.2, R48.2, R50.2, R52.2, R9.2, U18.AVCC, U18.VCC@1, U18.VCC@2, U19A.SCL, U19P.VCC, U2.3V3, U6A.SCL, U6P.VCC; no longer C10.1, C12.1, C4.1, J3.2, J5.2, J6.1, R10.2, R12.2, R13.2, R14.2, R15.2, R24.2, R25.2, R4.2, R6.2, U1.!RESET, U1.3V3OUT, U1.VCC, U1.VCCIO, U2.VCC, U5.OUT, U6.3V3
- net +5V: now also R13.1, R33.2; no longer C5.1, C6.1, C9.1, DIS1.VBIAS, J2.1, J3.1, J5.1, R11.2, U3.V+, U5.IN
- net D2_P: now also J5.D+, U22.USBDP; no longer R18.2, U1.USBDP
- net DTR: now also Q3.E, R7.2, U21.!DTR; no longer Q1.G, Q2.S, U1.!DTR
- net GND: now also C10.1, C13.2, C14.2, C17.1, C23.2, C31.2, C32.2, C33.2, C34.2, C35.2, D3.A, J4.5, J5.GND, J5.SHIELD, Q4.S, Q5.2, Q5.4, R11.1, R12.1, R57.1, SP1.P$2, SW3.1, SW4.1, SW5.1, U18.GND, U18.GND@1, U18.GND@2, U19A.G, U19P.GND, U2.GND-1, U2.GND-15, U2.GND-38, U2.GND-PAD, U21.GND, U21.GND@1, U21.GND@2, U21.GND@A, U21.TEST, U22.GND, U22.GND@1, U22.GND@2, U22.GND@A, U22.TEST, U6A.G, U6P.GND, U7.GND; no longer C10.2, C11.2, C17.2, C23.1, C24.1, D2.A, DIS1.GND, J2.2, J2.3, J3.7, J4.7, J5.7, J6.7, R1.1, R23.1, R9.1, SW3.P, SW3.P1, SW4.P, SW4.P1, SW5.P, SW5.P1, U1.GND@16, U1.GND@6, U2.GND, U6.GND1, U6.GND2
- net IO0: now also Q3.C, R6.2, U2.IO0; no longer C7.1, Q2.D, SW2.S, SW2.S1, U6.GPIO0
- net N$1: now also D3.C, R19.1, U5.COM, U7.COM; no longer R11.1, U3.ON/OFF
- net N$10: now also Q3.B, R8.1; no longer LED2.A, R13.1
- net N$18: now also D1.A, L1.3; no longer J5.6, U2.VFBLANK
- net N$19: now also Q1.G, U3.DR; no longer R23.2, U6.GPIO15
- net N$2: now also C27.1, U22.!RTS; no longer BATT1.+, J6.6
- net N$21: now also C11.2, R12.2; no longer R24.1, U6.EN
- net N$3: now also J3.1, U5.1C; no longer J5.3, U2.VFDIN
- net N$4: now also LED1.C, U21.CBUS1; no longer J5.4, U2.VFCLK
- net N$40: now also U5.4B, U6A.QE; no longer R1.2, U3.RT
- net N$41: now also U5.3B, U6A.QF; no longer D1.A, L1.2, U3.SW
- net N$43: now also U5.1B, U6A.QH; no longer R2.2, U3.FB
- net N$46: now also U19A.QB, U7.4B; no longer C13.1, R2.1
- net N$47: now also U19A.QC, U7.3B; no longer C13.2, C14.1, D2.C, R9.2, U3.IN-, VR1.A
- net N$48: now also U19A.QD, U7.2B; no longer C14.2, R7.2
- net N$5: now also LED2.C, U21.CBUS0; no longer J5.5, U2.VFLOAD
- net N$7: now also LED1.A, R1.1; no longer LED1.C, U1.CBUS1
- net N$8: now also LED2.A, R2.1; no longer LED2.C, U1.CBUS2
- net N$9: now also Q2.B, R7.1; no longer LED1.A, R12.1
- net RTS: now also Q2.E, R8.2, U21.!RTS; no longer Q1.S, Q2.G, U1.!RTS
- net RXD: now also U2.TXD0, U21.RXD; no longer U1.RXD, U6.TX
- net SCL: now also U2.IO22; no longer U6.GPIO14
- net SDA: now also U2.IO21; no longer U6.GPIO2
- net SQW: now also R9.1, U2.IO34; no longer R25.1, U6.GPIO13
- net SW3: now also R47.2, R48.1, U2.IO26; no longer J4.4, U6.GPIO7
- net SW4: now also R49.2, R50.1, U2.IO27; no longer J4.5, U6.GPIO6
- net TXD: now also U2.RXD0, U21.TXD; no longer U1.TXD, U6.RX
- net VBATT: now also BATT1.+; no longer J4.6
Other:
- note added: "desinged by Kinoshita"
- note added: "nixie tubes drive board"
- note removed: "5v 3.3v VFDIN VFCLK VFLOAD VFBLANK GND"
- note removed: "vfd tube drive board"
