File: circuit/vfd/vfd_drive.sch (EAGLE design)
At the start: 56 parts, among them J1 ZX62R-AB-5P, J2 DC_JACK_2DC0005D100, J3 PSM-210223-10, J4 PSM-210223-10, J5 FSM-21045-10, J6 FSM-21045-10, J7 PSM-210223-8, J8 FSM-21045-8, Q1 FA-238V, SW1 SKRPACE010, SW2 SKRPACE010, U1 PIC18F14K50-I, U2 MAX6921AWI+, U3 NJW4131, U4 DS3231M, U5 ADP3338AKCZ-3.3, U6 PSF-A85, U9 BME280

Commit message: [tem@]
Parts:
- removed C12: 10uF, taki-library:C-EUC3216
- removed J3, J4: PSM-210223-10, taki-library:PSM-210223-10
- removed J5, J6: FSM-21045-10, taki-library:FSM-21045-10
- removed J7: PSM-210223-8, taki-library:PSM-210223-8
- added R11: 27k, taki-library:R-EU_R0603
- C2: value 0.1uF -> 10uF; device taki-library:C-EUC0603 -> taki-library:C-EUC3216
Connections:
- removed net N$21: J5.3, U2.OUT0
- removed net N$22: J5.4, U2.OUT1
- removed net N$23: J5.5, U2.OUT2
- removed net N$24: J5.6, U2.OUT3
- removed net N$25: J5.7, U2.OUT4
- removed net N$26: J5.8, U2.OUT5
- removed net N$27: J5.9, U2.OUT6
- removed net N$28: J5.10, U2.OUT7
- removed net N$29: J6.2, U2.OUT8
- removed net N$30: J6.7, U2.OUT13
- removed net N$31: J6.8, U2.OUT12
- removed net N$32: J6.9, U2.OUT11
- removed net N$33: J6.10, U2.OUT10
- removed net N$34: J6.3, U2.OUT9
- removed net N$35: J6.6, U2.OUT14
- removed net N$36: J6.5, U2.OUT15
- removed net N$37: J6.4, U2.OUT16
- removed net N$38: J5.2, J7.2
- removed net N$7: J7.7, U2.VFBLANK
- net +24V: now also C2.1, U2.VBB; no longer C12.1
- net +5V: now also R11.2
- net GND: no longer C12.2, J3.1, J4.1, J5.1, J6.1, J7.8, U2.GND
- net N$1: now also R11.1, U3.ON/OFF; no longer J7.1, U2.VBB
- net N$2: no longer J7.3
- net N$3: no longer J7.4
- net N$39: no longer C2.1
- net N$4: no longer J7.5
- net N$5: no longer J7.6
- net VBIAS: no longer J4.2
- net VFD10: now also U2.OUT4; no longer J4.4
- net VFD11: now also U2.OUT5; no longer J4.5
- net VFD12: now also U2.OUT6; no longer J4.6
- net VFD14: now also U2.OUT7; no longer J4.7
- net VFD15: now also U2.OUT8; no longer J4.8
- net VFD16: now also U2.OUT9; no longer J4.9
- net VFD17: now also U2.OUT15; no longer J4.10
- net VFD18: now also U2.OUT14; no longer J3.10
- net VFD19: now also U2.OUT13; no longer J3.9
- net VFD2: now also U2.OUT16; no longer J3.5
- net VFD20: now also U2.OUT12; no longer J3.8
- net VFD21: now also U2.OUT11; no longer J3.7
- net VFD22: now also U2.OUT10; no longer J3.6
- net VFD3: now also U2.OUT0; no longer J3.4
- net VFD4: now also U2.OUT1; no longer J3.3
- net VFD5: now also U2.OUT2; no longer J3.2
- net VFD9: now also U2.OUT3; no longer J4.3
Other:
- moved on the sheet: C2
