File: circuit/vfd/vfd_drive.sch (EAGLE design)
At the start: 67 parts, among them J1 ZX62R-AB-5P, J2 2DC-0415D200, J3 FSM-21045-7, J5 PSM-210223-7, Q2 MMSS8050-L, Q3 MMSS8050-L, SW1 SKRPACE010, SW2 SKRPACE010, U1 FT231XS, U2 MAX6921AWI+, U3 NJW4131, U4 DS3231M, U5 ADP3338AKCZ-3.3, U6 PSF-A85, U9 BME280

Commit message: [complete]complete vfd driver board
Parts:
- removed LED4: VBUS, taki-library:LEDCHIPLED_0603
- removed Q3: MMSS8050-L, taki-library:MMSS8050-L
- removed R14: 1k, taki-library:R-EU_R0603
- removed R15: 4.7k, taki-library:R-EU_R0603
- removed R16, R19, R22: 10k, taki-library:R-EU_R0603
- removed R4, R6: 470, taki-library:R-EU_R0603
- added J4: PSM-210223-7, taki-library:PSM-210223-7
- added J6: FSM-21045-7, taki-library:FSM-21045-7
- added Q1: BSS138, taki-library:BSS138
- added R10, R25: 4.7k, taki-library:R-EU_R0603
- C10: value 1000pF -> 0.1uF
- Q2: value MMSS8050-L -> BSS138; device taki-library:MMSS8050-L -> taki-library:BSS138
Connections:
- removed net N$11: LED4.A, R14.1
- removed net N$12: C10.2, R6.1, SW2.S, SW2.S1
- removed net N$14: R15.1, R16.2, U1.CBUS0
- removed net N$15: Q2.B, R19.1
- removed net N$16: Q3.B, R22.1
- removed net N$2: C15.1, J5.2, U2.VCC
- removed net N$6: C8.2, R4.1, SW1.S, SW1.S1
- new net 32KHZ: R10.1, U4.32KHZ, U6.GPIO12
- new net SQW: R25.1, U4.SQW, U6.GPIO13
- new net SW1: J4.2
- new net SW2: J4.3
- new net SW3: J4.4
- new net SW4: J4.5
- new net VFBLANK: J3.6, U6.GPIO4
- new net VFCLK: J3.4, U6.GPIO10
- new net VFDIN: J3.3, U6.GPIO11
- new net VFLOAD: J3.5, U6.GPIO9
- net +3V3: now also C10.1, C15.1, J4.1, J5.2, J6.1, R10.2, R25.2, U2.VCC
- net DTR: now also Q1.G, Q2.S; no longer Q3.E, R19.2
- net GND: now also C10.2, J4.7, J6.7; no longer C10.1, C7.2, C8.1, LED4.C, R16.1, SW1.P, SW1.P1, SW2.P, SW2.P1
- net IO0: now also Q2.D; no longer Q3.C, R6.2
- net RESET: now also Q1.D; no longer C7.1, Q2.C, R4.2
- net RTS: now also Q1.S, Q2.G; no longer Q2.E, R22.2
- net SCL: now also U6.GPIO14
- net SDA: no longer U6.GPIO14
- net VBATT: now also J4.6
- net VBUS: no longer R14.2, R15.2
Other:
- note added: "5v 3.3v VFDIN VFCLK VFLOAD VFBLANK GND"
- moved on the sheet: BATT1, C1, C10, C11, C12, C13, C14, C15, C16, C17, C18, C19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

Commit message: [update] draw outline
Parts:
- added C20, C21, C23, C24: 1000pF, taki-library:C-EUC0603
- added R14, R15, R4, R6: 10k, taki-library:R-EU_R0603
- added SW3, SW4, SW5, SW6: JTP1230D, taki-library:JTP1230D
Connections:
- new net N$2: BATT1.+, J6.6
- new net SW1-SW: C20.2, J6.2, R4.1, SW3.S, SW3.S1
- new net SW2-SW: C21.2, J6.3, R6.1, SW4.S, SW4.S1
- new net SW3-SW: C23.2, J6.4, R14.1, SW5.S, SW5.S1
- new net SW4-SW: C24.2, J6.5, R15.1, SW6.S, SW6.S1
- net +3V3: now also R14.2, R15.2, R4.2, R6.2
- net GND: now also C20.1, C21.1, C23.1, C24.1, C7.2, C8.1, SW1.P, SW1.P1, SW2.P, SW2.P1, SW3.P, SW3.P1, SW4.P, SW4.P1, SW5.P, SW5.P1, SW6.P, SW6.P1
- net IO0: now also C7.1, SW2.S, SW2.S1
- net RESET: now also C8.2, SW1.S, SW1.S1
- net SW1: now also U6.GPIO5
- net SW2: now also U6.GPIO8
- net SW3: now also U6.GPIO7
- net SW4: now also U6.GPIO6
- net VBATT: no longer BATT1.+
Other:
- note added: "desgined by Kinoshita"
- note added: "vfd tube drive board"
- moved on the sheet: BATT1, C10, C7, C8, R23, R24, SW1, SW2, U6

Commit message: [add]add all
Parts:
- removed BATT1: SMTU2032, taki-library:SMTU2032
- removed C18, C19, C22: 0.1uF, taki-library:C-EUC0603
- removed C20, C21, C23, C24: 1000pF, taki-library:C-EUC0603
- removed D1: SS2040FL, taki-library:SS2040FL
- removed D2: BZX584C3V9, taki-library:BZX584C3V9
- removed J2: 2DC-0415D200, taki-library:2DC-0415D200
- removed J4: PSM-210223-7, taki-library:PSM-210223-7
- removed J6: FSM-21045-7, taki-library:FSM-21045-7
- removed LED1: RX, taki-library:LEDCHIPLED_0603
- removed LED2: TX, taki-library:LEDCHIPLED_0603
- removed R12, R13: 1k, taki-library:R-EU_R0603
- removed R14, R15, R23, R24, R4, R6: 10k, taki-library:R-EU_R0603
- removed R17, R18: 27, taki-library:R-EU_R0603
- removed R20, R21, R25: 4.7k, taki-library:R-EU_R0603
- removed SW1, SW2: SKRPACE010, taki-library:SKRPACE010
- removed SW3, SW4, SW5, SW6: JTP1230D, taki-library:JTP1230D
- removed U4: DS3231M, taki-library:DS3231M
- removed U9: BME280, taki-library:BME280
- added J7: DC_JACK_2DC0005D100, taki-library:DC_JACK_2DC0005D100
- added U8: ESP-WROOM-32, taki-library:ESP-WROOM-32
- C10: value 0.1uF -> 5uF
- C12: value 0.1uF -> 1500pF
- C13: value 10uF -> 680pF
- C14: value 270pF -> 100uF; device taki-library:C-EUC0603 -> taki-library:C-EUC1206
- C16: value 47pF -> 1uF
- C17: value 47pF -> 0.1uF
- C7: value 1000pF -> 1uF
- C8: value 1000pF -> 4.7uF
- L1: value NR10050T470M -> NR10050T221M; device taki-library:NR10050T470M -> taki-library:NR10050T221M
- R1: value 27k -> 220
- R10: value 4.7k -> 47k
- R11: value 27k -> 10k
- R2: value 8.2k -> 0.02; device taki-library:R-EU_R0603 -> taki-library:R-EU_R1206
- R7: value 27k -> 24k
- U1: value FT231XS -> CP2104; device taki-library:FT231XS -> taki-library:CP2104
- U3: value NJW4131 -> NJM2360AM; device taki-library:NJW4131 -> taki-library:NJM2360AM
- U6: value PSF-A85 -> RX8035LC; device ITEAD:PSF-A85 -> taki-library:RX8035LC
Connections:
- removed net 32KHZ: R10.1, U4.32KHZ, U6.GPIO12
- removed net D2_N: R17.2, U1.USBDM
- removed net D2_P: R18.2, U1.USBDP
- removed net D_N1: C16.1, J1.D-, R17.1
- removed net D_P1: C17.1, J1.D+, R18.1
- removed net N$10: LED2.A, R13.1
- removed net N$19: R23.2, U6.GPIO15
- removed net N$21: R24.1, U6.EN
- removed net N$40: R1.2, U3.RT
- removed net N$41: D1.A, L1.2, U3.SW
- removed net N$43: R2.2, U3.FB
- removed net N$46: C13.1, R2.1
- removed net N$47: C13.2, C14.1, D2.C, R9.2, U3.IN-, VR1.A
- removed net N$48: C14.2, R7.2
- removed net N$49: R8.2, VR1.E, VR1.S
- removed net RESET: C8.2, Q1.D, R3.1, SW1.S, SW1.S1, U6.RESET
- removed net RXD: U1.RXD, U6.TX
- removed net SQW: R25.1, U4.SQW, U6.GPIO13
- removed net SW1: J4.2, U6.GPIO5
- removed net SW1-SW: C20.2, J6.2, R4.1, SW3.S, SW3.S1
- removed net SW2: J4.3, U6.GPIO8
- removed net SW2-SW: C21.2, J6.3, R6.1, SW4.S, SW4.S1
- removed net SW3: J4.4, U6.GPIO7
- removed net SW3-SW: C23.2, J6.4, R14.1, SW5.S, SW5.S1
- removed net SW4: J4.5, U6.GPIO6
- removed net SW4-SW: C24.2, J6.5, R15.1, SW6.S, SW6.S1
- removed net TXD: U1.TXD, U6.RX
- removed net VBATT: J4.6, U4.VBAT
- new net D_N: J1.D-, U1.D-
- new net D_P: J1.D+, U1.D+
- new net EN: C12.1, Q1.D, R3.1, U8.EN
- new net ESP32_RX: U1.TXD, U8.TXD0
- new net ESP32_TX: U1.RXD, U8.RXD0
- new net N$11: C13.1, U3.CT
- new net N$12: R8.2, U3.INV, VR1.E, VR1.S
- new net N$13: R1.1, U3.CD
- new net N$14: L1.1, R1.2, R2.2, U3.SI
- new net N$6: L1.2, U3.CS
- net +24V: no longer D1.C, R7.1
- net +3V3: now also C14.1, C16.1, C7.1, R11.2, U1.REGIN, U1.VDD, U1.VIO, U6.VDD, U8.3V3; no longer C12.1, C18.1, C19.1, C22.1, J4.1, J6.1, R10.2, R12.2, R13.2, R14.2, R15.2, R20.2, R21.2, R24.2, R25.2, R4.2, R6.2, U1.!RESET, U1.3V3OUT, U1.VCC, U1.VCCIO, U4.VCC, U6.3V3, U9.!CS, U9.SDO/ADR, U9.VDD, U9.VDDIO
- net +5V: now also J7.1, R2.1, U3.VDD; no longer J2.1, L1.1, R11.2, U3.V+
- net DTR: now also U1.DTR; no longer U1.!DTR
- net GND: now also C13.2, C14.2, C8.2, J7.2, J7.3, R10.1, U1.GND, U3.ES, U3.GND, U8.GND-1, U8.GND-15, U8.GND-38, U8.GND-PAD; no longer BATT1.-, C18.2, C19.2, C20.1, C21.1, C22.2, C23.1, C24.1, C8.1, D2.A, J2.2, J2.3, J4.7, J6.7, R1.1, R23.1, SW1.P, SW1.P1, SW2.P, SW2.P1, SW3.P, SW3.P1, SW4.P, SW4.P1, SW5.P, SW5.P1, SW6.P, SW6.P1, U1.GND@16, U1.GND@6, U3.AGND, U3.PGND, U4.GND, U6.GND1, U6.GND2, U9.GND
- net IO0: now also U8.IO0; no longer C7.1, SW2.S, SW2.S1, U6.GPIO0
- net N$1: now also R9.2, VR1.A; no longer R11.1, U3.ON/OFF
- net N$2: now also C17.1, U6.VOUT; no longer BATT1.+, J6.6
- net N$7: now also R11.1, U1.RST; no longer LED1.C, U1.CBUS1
- net N$8: now also R10.2, R7.1, U1.VBUS; no longer LED2.C, U1.CBUS2
- net N$9: now also C8.1, U1.VPP; no longer LED1.A, R12.1
- net RTS: now also U1.RTS; no longer U1.!RTS
- net SCL: now also U6.SCL, U8.IO22; no longer R20.1, U4.SCL, U6.GPIO14, U9.SCK/SCL
- net SDA: now also U6.SDA, U8.IO21; no longer R21.1, U4.SDA, U6.GPIO2, U9.SDI/SDA
- net VBUS: now also R7.2
- net VFBLANK: no longer U6.GPIO4
- net VFCLK: no longer U6.GPIO10
- net VFDIN: no longer U6.GPIO11
- net VFLOAD: no longer U6.GPIO9
Other:
- moved on the sheet: C10, C12, C13, C14, C16, C17, C3, C4, C5, C6, C7, C8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

Commit message: [add]add all
Parts:
- removed U6: RX8035LC, taki-library:RX8035LC
- added C18: UWT1E221MNL1GS, taki-library:UWT1E221MNL1GS
- added C19, C20, C21, C22: 0.1uF, taki-library:C-EUC0603
- added D1: MS18F, taki-library:MS18F
- added J2: FSM-21045-7, taki-library:FSM-21045-7
- added J4: PSM-210223-7, taki-library:PSM-210223-7
- added Q3, Q4, Q5, Q6: BSS138, taki-library:BSS138
- added R12, R14, R15, R17, R20, R21, R4, R6: 10k, taki-library:R-EU_R0603
- added R13, R16, R18, R19: 1k, taki-library:R-EU_R0603
- added SP1: PKLCS1212E4001-R1, taki-library:PKLCS1212E4001-R1
- added SW1: AT407, taki-library:AT407
- added U4: HV5812SOW, taki-library:HV5812SOW
- C13: value 680pF -> 470pF
- C15: value 0.1uF -> (none); device taki-library:C-EUC0603 -> taki-library:CPOL-EUSE-5R5-D155VY
- R2: value 0.02 -> 0.2
- R8: value 3.3k -> 220k
- R9: value 3.3k -> 8.2k
- U2: value MAX6921AWI+ -> RX8900CE; device taki-library:MAX6921AWI+ -> taki-library:RX8900CE
Connections:
- removed net N$18: J5.6, U2.VFBLANK
- removed net VFBLANK: J3.6
- removed net VFCLK: J3.4
- removed net VFDIN: J3.3
- removed net VFLOAD: J3.5
- new net BATT: J4.4, R6.2
- new net BL: J5.2, U4.BLANKING
- new net CLK: J5.5, U4.CLK
- new net DATA: J5.4, U4.DIN
- new net EDLC: C15.+, J2.4
- new net ESP32_BL: R13.2, U8.IO19
- new net ESP32_CLK: R19.2, U8.IO5
- new net ESP32_DATA: R18.2, U8.IO18
- new net ESP32_STR: R16.2, U8.IO17
- new net INT: R21.1, U2.INT, U8.IO4
- new net N$10: R4.1, SP1.1
- new net N$15: Q5.G, R18.1
- new net SP: R4.2, U8.IO13
- new net STR: J5.6, U4.STROBE
- new net SW: R12.1, SW1.1
- new net VFD_BL: J3.2, Q4.D, R14.1
- new net VFD_CLK: J3.5, Q6.D, R20.1
- new net VFD_DATA: J3.4, Q5.D, R17.1
- new net VFD_STR: J3.6, Q3.D, R15.1
- net +24V: now also C20.1, D1.C, J2.3, J3.3, J4.3, J5.3, U4.VPP; no longer U2.VBB
- net +3V3: now also C22.1, J2.2, J4.2, R12.2, R21.2, U2.VDD; no longer C15.1, J3.2, J5.2, U2.VCC, U6.VDD
- net +5V: now also C17.1, C18.+, C19.1, J2.7, J3.7, J4.7, J5.7, R14.2, R15.2, R17.2, R20.2, U4.VDD; no longer J3.1, J5.1
- net GND: now also C15.-, C18.-, C19.2, C20.2, C21.2, C22.2, J2.1, J3.1, J4.1, J5.1, Q3.S, Q4.S, Q5.S, Q6.S, SP1.P$2, SW1.2, U2.FOE, U4.GND; no longer C15.2, J3.7, J5.7
- net N$1: now also VR1.E, VR1.S; no longer VR1.A
- net N$12: now also VR1.A; no longer VR1.E, VR1.S
- net N$2: now also Q4.G, R13.1; no longer C17.1, U6.VOUT
- net N$3: now also Q6.G, R19.1; no longer J5.3, U2.VFDIN
- net N$4: now also Q3.G, R16.1; no longer J5.4, U2.VFCLK
- net N$5: now also C21.1, R6.1, U2.VBAT; no longer J5.5, U2.VFLOAD
- net N$6: now also D1.A
- net SCL: now also U2.SCL; no longer U6.SCL
- net SDA: now also U2.SDA; no longer U6.SDA
- net VFD10: now also U4.HVOUT7; no longer U2.OUT4
- net VFD11: now also U4.HVOUT6; no longer U2.OUT5
- net VFD12: now also U4.HVOUT5; no longer U2.OUT6
- net VFD14: now also U4.HVOUT12; no longer U2.OUT8
- net VFD15: now also U4.HVOUT13; no longer U2.OUT9
- net VFD16: now also U4.HVOUT14; no longer U2.OUT16
- net VFD17: now also U4.HVOUT15; no longer U2.OUT15
- net VFD18: now also U4.HVOUT16; no longer U2.OUT14
- net VFD19: now also U4.HVOUT17; no longer U2.OUT13
- net VFD2: now also U4.HVOUT4; no longer U2.OUT7
- net VFD20: now also U4.HVOUT18; no longer U2.OUT12
- net VFD21: now also U4.HVOUT19; no longer U2.OUT11
- net VFD22: now also U4.HVOUT20; no longer U2.OUT10
- net VFD3: now also U4.HVOUT3; no longer U2.OUT0
- net VFD4: now also U4.HVOUT2; no longer U2.OUT1
- net VFD5: now also U4.HVOUT1; no longer U2.OUT2
- net VFD9: now also U4.HVOUT8; no longer U2.OUT3
Other:
- note removed: "5v 3.3v VFDIN VFCLK VFLOAD VFBLANK GND"
- moved on the sheet: C10, C11, C12, C13, C14, C16, C17, C2, C3, C4, C5, C6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
